Commit message: Merged duplicated package guardian_description.

File: guardian_sim/guardian_description/urdf/gball_ita.urdf (robot description, URDF)
Before this commit: robot gball, 22 links, 21 joints
Links:
- link back_left_wheel: geometry collision mesh filename=package://guardian_description/meshes/wheel.stl; visual mesh filename=package://guardian_description/meshes/wheel.stl
- link back_right_wheel: geometry collision mesh filename=package://guardian_description/meshes/wheel.stl; visual mesh filename=package://guardian_description/meshes/wheel.stl
- link base_link: geometry collision mesh filename=package://guardian_description/meshes/chassis/v6/chassisV6.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; visual mesh filename=package://guardian_description/meshes/chassis/v6/chassisV6.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
- link front_left_wheel: geometry collision mesh filename=package://guardian_description/meshes/wheel.stl; visual mesh filename=package://guardian_description/meshes/wheel.stl
- link front_right_wheel: geometry collision mesh filename=package://guardian_description/meshes/wheel.stl; visual mesh filename=package://guardian_description/meshes/wheel.stl
- link left_track: geometry collision mesh filename=package://guardian_description/meshes/others/v5/trackV5_l.s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; visual mesh filename=package://guardian_description/meshes/others/v5/trackV5_l.s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
- link right_track: geometry collision mesh filename=package://guardian_description/meshes/others/v5/trackV5_l.s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; visual mesh filename=package://guardian_description/meshes/others/v5/trackV5_l.s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

File: guardian_sim/guardian_description/urdf/gball_ita_23082013.urdf (robot description, URDF)
Before this commit: robot gball, 22 links, 21 joints
Links:
- link back_left_wheel: geometry collision mesh filename=package://guardian_description/meshes/wheel.stl; visual mesh filename=package://guardian_description/meshes/wheel.stl
- link back_right_wheel: geometry collision mesh filename=package://guardian_description/meshes/wheel.stl; visual mesh filename=package://guardian_description/meshes/wheel.stl
- link base_link: geometry collision mesh filename=package://guardian_description/meshes/chassis/v6/chassisV6.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; visual mesh filename=package://guardian_description/meshes/chassis/v6/chassisV6.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
- link front_left_wheel: geometry collision mesh filename=package://guardian_description/meshes/wheel.stl; visual mesh filename=package://guardian_description/meshes/wheel.stl
- link front_right_wheel: geometry collision mesh filename=package://guardian_description/meshes/wheel.stl; visual mesh filename=package://guardian_description/meshes/wheel.stl
- link left_track: geometry collision mesh filename=package://guardian_description/meshes/others/v5/trackV5_l.s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; visual mesh filename=package://guardian_description/meshes/others/v5/trackV5_l.s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
- link right_track: geometry collision mesh filename=package://guardian_description/meshes/others/v5/trackV5_l.s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; visual mesh filename=package://guardian_description/meshes/others/v5/trackV5_l.s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

File: guardian_sim/guardian_description/urdf/gball_ita_sinfootprint.urdf (robot description, URDF)
Before this commit: robot gball, 21 links, 20 joints
Links:
- link back_left_wheel: geometry collision mesh filename=package://guardian_description/meshes/wheel.stl; visual mesh filename=package://guardian_description/meshes/wheel.stl
- link back_right_wheel: geometry collision mesh filename=package://guardian_description/meshes/wheel.stl; visual mesh filename=package://guardian_description/meshes/wheel.stl
- link base_link: geometry collision mesh filename=package://guardian_description/meshes/chassis/v6/chassisV6.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; visual mesh filename=package://guardian_description/meshes/chassis/v6/chassisV6.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
- link front_left_wheel: geometry collision mesh filename=package://guardian_description/meshes/wheel.stl; visual mesh filename=package://guardian_description/meshes/wheel.stl
- link front_right_wheel: geometry collision mesh filename=package://guardian_description/meshes/wheel.stl; visual mesh filename=package://guardian_description/meshes/wheel.stl
- link left_track: geometry collision mesh filename=package://guardian_description/meshes/others/v5/trackV5_l.s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; visual mesh filename=package://guardian_description/meshes/others/v5/trackV5_l.s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
- link right_track: geometry collision mesh filename=package://guardian_description/meshes/others/v5/trackV5_l.s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; visual mesh filename=package://guardian_description/meshes/others/v5/trackV5_l.s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

File: guardian_sim/guardian_description/urdf/guardian.urdf (robot description, URDF)
Before this commit: robot guardian, 11 links, 10 joints
Links:
- link back_left_wheel: geometry collision mesh filename=package://guardian_description/meshes/wheel.stl; visual mesh filename=package://guardian_description/meshes/wheel.stl
- link back_right_wheel: geometry collision mesh filename=package://guardian_description/meshes/wheel.stl; visual mesh filename=package://guardian_description/meshes/wheel.stl
- link base_link: geometry collision mesh filename=package://guardian_description/meshes/chassis/v6/chassisV6.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; visual mesh filename=package://guardian_description/meshes/chassis/v6/chassisV6.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
- link front_left_wheel: geometry collision mesh filename=package://guardian_description/meshes/wheel.stl; visual mesh filename=package://guardian_description/meshes/wheel.stl
- link front_right_wheel: geometry collision mesh filename=package://guardian_description/meshes/wheel.stl; visual mesh filename=package://guardian_description/meshes/wheel.stl
- link left_track: geometry collision mesh filename=package://guardian_description/meshes/others/v5/trackV5_l.s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; visual mesh filename=package://guardian_description/meshes/others/v5/trackV5_l.s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
- link right_track: geometry collision mesh filename=package://guardian_description/meshes/others/v5/trackV5_l.s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; visual mesh filename=package://guardian_description/meshes/others/v5/trackV5_l.s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

File: guardian_sim/guardian_description/urdf/guardian_ita.urdf (robot description, URDF)
Before this commit: robot gball, 11 links, 10 joints
Links:
- link back_left_wheel: geometry collision mesh filename=package://guardian_description/meshes/wheel.stl; visual mesh filename=package://guardian_description/meshes/wheel.stl
- link back_right_wheel: geometry collision mesh filename=package://guardian_description/meshes/wheel.stl; visual mesh filename=package://guardian_description/meshes/wheel.stl
- link base_link: geometry collision mesh filename=package://guardian_description/meshes/chassis/v6/chassisV6.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; visual mesh filename=package://guardian_description/meshes/chassis/v6/chassisV6.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
- link front_left_wheel: geometry collision mesh filename=package://guardian_description/meshes/wheel.stl; visual mesh filename=package://guardian_description/meshes/wheel.stl
- link front_right_wheel: geometry collision mesh filename=package://guardian_description/meshes/wheel.stl; visual mesh filename=package://guardian_description/meshes/wheel.stl
- link left_track: geometry collision mesh filename=package://guardian_description/meshes/others/v5/trackV5_l.s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; visual mesh filename=package://guardian_description/meshes/others/v5/trackV5_l.s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
- link right_track: geometry collision mesh filename=package://guardian_description/meshes/others/v5/trackV5_l.s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; visual mesh filename=package://guardian_description/meshes/others/v5/trackV5_l.s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

File: guardian_sim/guardian_description/urdf/gwam_ume.urdf (robot description, URDF)
Before this commit: robot gwam, 18 links, 17 joints
Links:
- link back_left_wheel: geometry collision mesh filename=package://guardian_description/meshes/wheel.stl; visual mesh filename=package://guardian_description/meshes/wheel.stl
- link back_right_wheel: geometry collision mesh filename=package://guardian_description/meshes/wheel.stl; visual mesh filename=package://guardian_description/meshes/wheel.stl
- link base_link: geometry collision mesh filename=package://guardian_description/meshes/chassis/v5/chassisV5_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; visual mesh filename=package://guardian_description/meshes/chassis/v5/chassisV5_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
- link front_left_wheel: geometry collision mesh filename=package://guardian_description/meshes/wheel.stl; visual mesh filename=package://guardian_description/meshes/wheel.stl
- link front_right_wheel: geometry collision mesh filename=package://guardian_description/meshes/wheel.stl; visual mesh filename=package://guardian_description/meshes/wheel.stl
- link left_track: geometry collision mesh filename=package://guardian_description/meshes/others/v5/trackV5_l.s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; visual mesh filename=package://guardian_description/meshes/others/v5/trackV5_l.s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
- link right_track: geometry collision mesh filename=package://guardian_description/meshes/others/v5/trackV5_l.s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; visual mesh filename=package://guardian_description/meshes/others/v5/trackV5_l.s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
- link wam_link1: geometry collision mesh filename=package://guardian_description/meshes/wam1.stl scale=1.0 1.0 1.0; visual mesh filename=package://guardian_description/meshes/wam1.stl scale=1.0 1.0 1.0
- link wam_link2: geometry collision mesh filename=package://guardian_description/meshes/wam2.stl scale=1.0 1.0 1.0; visual mesh filename=package://guardian_description/meshes/wam2.stl scale=1.0 1.0 1.0
- link wam_link3: geometry collision mesh filename=package://guardian_description/meshes/wam3.stl scale=1.0 1.0 1.0; visual mesh filename=package://guardian_description/meshes/wam3.stl scale=1.0 1.0 1.0
- link wam_link4: geometry collision mesh filename=package://guardian_description/meshes/wam4.stl scale=1.0 1.0 1.0; visual mesh filename=package://guardian_description/meshes/wam4.stl scale=1.0 1.0 1.0
- link wam_link5: geometry collision mesh filename=package://guardian_description/meshes/wam5.stl scale=1.0 1.0 1.0; visual mesh filename=package://guardian_description/meshes/wam5.stl scale=1.0 1.0 1.0
- link wam_link6: geometry collision mesh filename=package://guardian_description/meshes/wam6.stl scale=1.0 1.0 1.0; visual mesh filename=package://guardian_description/meshes/wam6.stl scale=1.0 1.0 1.0
- link wam_link7: geometry collision mesh filename=package://guardian_description/meshes/wam7.stl scale=1.0 1.0 1.0; visual mesh filename=package://guardian_description/meshes/wam7.stl scale=1.0 1.0 1.0
