Commit message: CAD world and tilt laser
Bug fixes:
#1774
#1807
#1806

Tilt laser joystick - working, but slow

File: guardian_sim/guardian_description/urdf/guardian.urdf.xacro (robot description, xacro)
@@ -92,8 +92,4 @@
     </collision>
   </link>
-  <gazebo reference="left_track">
-    <material>Gazebo/FlatBlack</material>
-    <turnGravityOff>false</turnGravityOff>
-  </gazebo>
   <joint name="joint_left_track" type="fixed">
     <parent link="base_link"/>
@@ -124,8 +120,4 @@
     </collision>
   </link>
-  <gazebo reference="right_track">
-    <material>Gazebo/FlatBlack</material>
-    <turnGravityOff>false</turnGravityOff>
-  </gazebo>
   <joint name="joint_right_track" type="fixed">
     <parent link="base_link"/>
@@ -141,5 +133,5 @@
     </inertial>
     <visual>
-       <origin xyz="0 0 0" rpy="0 0 3.1416" />
+       <origin xyz="0 0 0" rpy="0 0 ${PI}" /> <!-- 3.1416 -->
        <geometry>
 	 <mesh filename="package://guardian_description/meshes/wheel.dae"/>
@@ -150,5 +142,5 @@
     </visual>
     <collision>
-       <origin xyz="0 0 0" rpy="0 0 3.1416" />
+       <origin xyz="0 0 0" rpy="0 0 ${PI}" />
        <geometry>
          <mesh filename="package://guardian_description/meshes/wheel.dae"/>
@@ -223,5 +215,5 @@
     </inertial>
     <visual>
-       <origin xyz="0 0 0" rpy="0 0 3.1416" />
+       <origin xyz="0 0 0" rpy="0 0 ${PI}" />
        <geometry>
          <mesh filename="package://guardian_description/meshes/wheel.dae"/>
@@ -232,5 +224,5 @@
     </visual>
     <collision>
-       <origin xyz="0 0 0" rpy="0 0 3.1416" />
+       <origin xyz="0 0 0" rpy="0 0 ${PI}" />
        <geometry>
          <mesh filename="package://guardian_description/meshes/wheel.dae"/>
@@ -299,5 +291,5 @@
   </transmission>
 	<!-- KINECT CAMERA -->
-  <joint name="camera_joint" type="fixed">
+  <!--joint name="camera_joint" type="fixed">
      <axis xyz="0 1 0" />
      <origin xyz="0.5 0 0.31"/>
@@ -311,9 +303,64 @@
        <inertia ixx="0.0001" ixy="0" ixz="0" iyy="0.000001" iyz="0" izz="0.0001" />
     </inertial>
-  </link>
+  </link-->
+<!-- AXIS PTZ CAMERA WITH PAN AND TILT -->
+  <!--link name="hokuyo_laser_tilt_link">
+     <inertial>
+       <mass value="0.1" />
+       <origin xyz="0 0 0" rpy="0 0 0" />
+       <inertia ixx="0.1" ixy="0" ixz="0" iyy="0.1" iyz="0" izz="0.1" />
+    </inertial>
+  </link-->
+  <joint name="laser_tilt_joint" type="revolute">
+     <axis xyz="0 1 0" />
+     <!--origin xyz="0.180 0.0 0.270"/-->
+     <origin xyz="0.5 0 0.31" rpy="0 0.52 0" />
+     <parent link="base_link"/>
+     <child link="hokuyo_laser_tilt_link"/>
+     <limit effort="${ptz_joint_effort_limit}" velocity="${ptz_joint_velocity_limit}" lower="-1.5708" upper="1.5708"/>
+     <joint_properties damping="${ptz_joint_damping}" friction="{ptz_joint_friction}"/>
+  </joint>
+  <link name="hokuyo_laser_tilt_link">
+     <inertial>
+       <mass value="0.1" />
+       <origin xyz="0 0 0" rpy="0 0 0" />
+       <inertia ixx="0.1" ixy="0" ixz="0" iyy="0.1" iyz="0" izz="0.1" />
+    </inertial>
+    <visual>
+        <origin xyz="0 0 0" rpy="0 0 0" />
+        <geometry>
+          <mesh filename="package://pr2_description/meshes/tilting_laser_v0/tilting_hokuyo.dae" />
+          <!--mesh filename="package://guardian_description/meshes/hokuyo-utm30-lx.dae"/-->
+        </geometry>
+        <material name="Red" />
+      </visual>
+      <collision>
+        <origin xyz="0 0 0" rpy="0 0 0" />
+        <geometry>
+          <mesh filename="package://pr2_description/meshes/tilting_laser_v0/tilting_hokuyo_L.stl" />
+          <!--mesh filename="package://guardian_description/meshes/hokuyo-utm30-lx.dae"/-->
+        </geometry>
+      </collision>
+  </link>
+  <!--joint name="joint_laser_tilt" type="continuous">
+     <axis xyz="0 1 0" />
+     <origin xyz="0.0 0.0 0.0"/>
+     <parent link="hokuyo_laser_tilt_link"/>
+     <child link="laser_tilt_link"/>
+     <limit effort="${ptz_joint_effort_limit}" velocity="${ptz_joint_velocity_limit}" lower="-1.5708" upper="1.5708"/>
+     <joint_properties damping="${ptz_joint_damping}" friction="{ptz_joint_friction}"/>
+  </joint-->
+  <transmission name="joint_laser_tilt_trans">
+   <type>transmission_interface/SimpleTransmission</type>
+     <joint name="laser_tilt_joint" />
+     <actuator name="laser_tilt_motor">
+     <hardwareInterface>EffortJointInterface</hardwareInterface>
+       <mechanicalReduction>${ptz_mechanical_reduction}</mechanicalReduction>
+     </actuator>
+  </transmission>
   <!-- HOKUYO SENSOR -->
   <joint name="hokuyo_laser_joint" type="fixed">
      <axis xyz="0 1 0" />
-     <origin xyz="0.5 0 0.31"/>
+     <origin xyz="-0.4 0 0.31" rpy="0 0 ${PI}" />
      <parent link="base_link"/>
      <child link="hokuyo_laser_link"/>
@@ -327,10 +374,10 @@
       </geometry>
     </collision>
-    <!-- visual>
+    <visual>
       <origin xyz="0 0 0" rpy="0 0 0"/>
       <geometry>
         <mesh filename="package://guardian_description/meshes/hokuyo-utm30-lx.dae"/>
       </geometry>
-    </visual -->
+    </visual>
     <inertial>
       <mass value="1e-5" />

Commit message: Guardian ship interior, minor laser fixes
CAD related files were not on last commit and were now renamed to
ship_interior.

Lasers were updated to match datasheet. 

Tilt laser with joystick command and tilit limit #1820

File: guardian_sim/guardian_description/urdf/guardian.urdf.xacro (robot description, xacro)
@@ -315,5 +315,5 @@
      <axis xyz="0 1 0" />
      <!--origin xyz="0.180 0.0 0.270"/-->
-     <origin xyz="0.5 0 0.31" rpy="0 0.52 0" />
+     <origin xyz="0.5 0 0.31" rpy="0 0 ${PI}" />
      <parent link="base_link"/>
      <child link="hokuyo_laser_tilt_link"/>
@@ -327,17 +327,17 @@
        <inertia ixx="0.1" ixy="0" ixz="0" iyy="0.1" iyz="0" izz="0.1" />
     </inertial>
-    <visual>
+    <!--visual>
         <origin xyz="0 0 0" rpy="0 0 0" />
-        <geometry>
-          <mesh filename="package://pr2_description/meshes/tilting_laser_v0/tilting_hokuyo.dae" />
-          <!--mesh filename="package://guardian_description/meshes/hokuyo-utm30-lx.dae"/-->
+        <geometry-->
+          <!--mesh filename="package://pr2_description/meshes/tilting_laser_v0/tilting_hokuyo.dae" /-->
+          <!--mesh filename="package://guardian_description/meshes/hokuyo-utm30-lx.dae"/>
         </geometry>
         <material name="Red" />
-      </visual>
+      </visual-->
       <collision>
         <origin xyz="0 0 0" rpy="0 0 0" />
         <geometry>
-          <mesh filename="package://pr2_description/meshes/tilting_laser_v0/tilting_hokuyo_L.stl" />
-          <!--mesh filename="package://guardian_description/meshes/hokuyo-utm30-lx.dae"/-->
+          <!--mesh filename="package://pr2_description/meshes/tilting_laser_v0/tilting_hokuyo_L.stl" /-->
+          <mesh filename="package://guardian_description/meshes/hokuyo-utm30-lx.dae"/>
         </geometry>
       </collision>

Commit message: Tilt Laser frame bug fix, ship_interior map
Tilt Laser bug fix : #1824
added ship interior map to guardian_navigation
guardian_office.launch updated to not duplicate code from
guardian.launch

File: guardian_sim/guardian_description/urdf/guardian.urdf.xacro (robot description, xacro)
@@ -315,5 +315,5 @@
      <axis xyz="0 1 0" />
      <!--origin xyz="0.180 0.0 0.270"/-->
-     <origin xyz="0.5 0 0.31" rpy="0 0 ${PI}" />
+     <origin xyz="0.5 0 0.31" rpy="0 0 0" />
      <parent link="base_link"/>
      <child link="hokuyo_laser_tilt_link"/>

Commit message: guardian_robot_control and laser fix
guardian_robot_control - cmd_vel topic is not hardcoded, but param
lasers 

laser - new angles....

File: guardian_sim/guardian_description/urdf/guardian.urdf.xacro (robot description, xacro)
@@ -304,12 +304,5 @@
     </inertial>
   </link-->
-<!-- AXIS PTZ CAMERA WITH PAN AND TILT -->
-  <!--link name="hokuyo_laser_tilt_link">
-     <inertial>
-       <mass value="0.1" />
-       <origin xyz="0 0 0" rpy="0 0 0" />
-       <inertia ixx="0.1" ixy="0" ixz="0" iyy="0.1" iyz="0" izz="0.1" />
-    </inertial>
-  </link-->
+  <!-- FRONT - TILT LASER -->
   <joint name="laser_tilt_joint" type="revolute">
      <axis xyz="0 1 0" />
@@ -362,5 +355,5 @@
   <joint name="hokuyo_laser_joint" type="fixed">
      <axis xyz="0 1 0" />
-     <origin xyz="-0.4 0 0.31" rpy="0 0 ${PI}" />
+     <origin xyz="-0.55 0 0.31" rpy="0 0 ${PI}" />
      <parent link="base_link"/>
      <child link="hokuyo_laser_link"/>

Commit message: guardian robot control - wheels and tilt separation
guardian_robot_control - doesn't command wheels nor pubs wheels' joints,
now only commnads tilt laser. All topics subscribed are now params
(yaml).

guardian_control - wheels' controllers deleted

guardian.gazebo, guardian.urdf.xacro - camera was commented out.

File: guardian_sim/guardian_description/urdf/guardian.urdf.xacro (robot description, xacro)
@@ -406,5 +406,5 @@
   </link>
   <!-- AXIS PTZ CAMERA WITH PAN AND TILT -->
-  <link name="camera_base_link">
+  <!-- link name="camera_base_link">
      <inertial>
        <mass value="0.1" />
@@ -464,4 +464,4 @@
        <mechanicalReduction>${ptz_mechanical_reduction}</mechanicalReduction>
      </actuator>
-  </transmission>
+  </transmission-->
 </robot>

Commit message: Guardian two lasers
guardian2lasers.dae & .stl added to meshes folder
guardian chassis updated to guardian2lasers in guardian.urdf.xacro
lasers positions updated
laser collision fixed #1770

File: guardian_sim/guardian_description/urdf/guardian.urdf.xacro (robot description, xacro)
@@ -59,5 +59,5 @@
        <origin xyz="0 0 0" rpy="0 0 0" />
        <geometry>
-	 <mesh filename="package://guardian_description/meshes/chassis/v6/chassisV6.dae"/>
+	     <mesh filename="package://guardian_description/meshes/chassis/two_lasers/guardian2lasers.dae"/>
        </geometry>
     </visual>
@@ -65,5 +65,5 @@
        <origin xyz="0 0 0" rpy="0 0 0 " />
        <geometry>
-         <mesh filename="package://guardian_description/meshes/chassis/v6/chassisV6.dae"/>
+         <mesh filename="package://guardian_description/meshes/chassis/two_lasers/guardian2lasers.dae"/>
        </geometry>
     </collision>
@@ -308,5 +308,5 @@
      <axis xyz="0 1 0" />
      <!--origin xyz="0.180 0.0 0.270"/-->
-     <origin xyz="0.5 0 0.31" rpy="0 0 0" />
+     <origin xyz="0.48856 0 0.24" rpy="0 0 0" /> <!-- 0.1885 --><!--   <origin xyz="0.5 0 0.31" rpy="0 0 0" /> -->
      <parent link="base_link"/>
      <child link="hokuyo_laser_tilt_link"/>
@@ -328,20 +328,11 @@
         <material name="Red" />
       </visual-->
-      <collision>
+      <!-- collision>
         <origin xyz="0 0 0" rpy="0 0 0" />
         <geometry>
-          <!--mesh filename="package://pr2_description/meshes/tilting_laser_v0/tilting_hokuyo_L.stl" /-->
           <mesh filename="package://guardian_description/meshes/hokuyo-utm30-lx.dae"/>
         </geometry>
-      </collision>
-  </link>
-  <!--joint name="joint_laser_tilt" type="continuous">
-     <axis xyz="0 1 0" />
-     <origin xyz="0.0 0.0 0.0"/>
-     <parent link="hokuyo_laser_tilt_link"/>
-     <child link="laser_tilt_link"/>
-     <limit effort="${ptz_joint_effort_limit}" velocity="${ptz_joint_velocity_limit}" lower="-1.5708" upper="1.5708"/>
-     <joint_properties damping="${ptz_joint_damping}" friction="{ptz_joint_friction}"/>
-  </joint-->
+      </collision-->
+  </link>
   <transmission name="joint_laser_tilt_trans">
    <type>transmission_interface/SimpleTransmission</type>
@@ -355,5 +346,5 @@
   <joint name="hokuyo_laser_joint" type="fixed">
      <axis xyz="0 1 0" />
-     <origin xyz="-0.55 0 0.31" rpy="0 0 ${PI}" />
+     <origin xyz="-0.43235 0 0.3" rpy="0 0 ${PI}" /> <!--  z: 0.24199 --> <!-- <origin xyz="-0.55 0 0.31" rpy="0 0 ${PI}" /> -->
      <parent link="base_link"/>
      <child link="hokuyo_laser_link"/>
@@ -361,5 +352,5 @@
   <!-- Hokuyo Laser -->
   <link name="hokuyo_laser_link">
-    <collision>
+    <!--  collision>
       <origin xyz="0 0 0" rpy="0 0 0"/>
       <geometry>
@@ -372,5 +363,5 @@
         <mesh filename="package://guardian_description/meshes/hokuyo-utm30-lx.dae"/>
       </geometry>
-    </visual>
+    </visual-->
     <inertial>
       <mass value="1e-5" />

Commit message: laser_tilt_command - find tilt index
comments on guardian urdfs for better separation of various parts

File: guardian_sim/guardian_description/urdf/guardian.urdf.xacro (robot description, xacro)
@@ -69,4 +69,5 @@
     </collision>
   </link>
+<!-- ################# TRACKS ################# -->
   <!-- LEFT TRACK (BLACK) -->
   <link name="left_track">
@@ -125,4 +126,5 @@
     <origin xyz="0.0 0.0 0.0" rpy="0 0 3.1415926535" />
   </joint>
+<!-- ################# WHEELS ################# -->
   <!-- BACK LEFT WHEEL (GREY) -->
   <link name="back_left_wheel">
@@ -290,4 +292,5 @@
      <!-- motorTorqueConstant>1</motorTorqueConstant -->
   </transmission>
+<!-- ################# SENSORS ################# -->
   <!-- FRONT - TILT LASER - URG-04LX -->
   <joint name="hokuyo_tilt_laser_joint" type="revolute">
@@ -382,63 +385,3 @@
       </collision>
   </link>
-  <!-- AXIS PTZ CAMERA WITH PAN AND TILT -->
-  <!-- link name="camera_base_link">
-     <inertial>
-       <mass value="0.1" />
-       <origin xyz="0 0 0" rpy="0 0 0" />
-       <inertia ixx="0.1" ixy="0" ixz="0" iyy="0.1" iyz="0" izz="0.1" />
-    </inertial>
-  </link>
-  <joint name="joint_camera" type="fixed">
-     <axis xyz="0 1 0" />
-     <origin xyz="0.180 0.0 0.270"/>
-     <parent link="base_link"/>
-     <child link="camera_base_link"/>
-  </joint>
-  <link name="camera_pan_link">
-     <inertial>
-       <mass value="0.1" />
-       <origin xyz="0 0 0" rpy="0 0 0" />
-       <inertia ixx="0.1" ixy="0" ixz="0" iyy="0.1" iyz="0" izz="0.1" />
-    </inertial>
-  </link>
-  <joint name="joint_camera_pan" type="continuous">
-     <axis xyz="0 0 1" />
-     <origin xyz="0.0 0.0 0.0"/>
-     <parent link="camera_base_link"/>
-     <child link="camera_pan_link"/>
-     <limit effort="${ptz_joint_effort_limit}" velocity="${ptz_joint_velocity_limit}" lower="-3.1416" upper="3.1416"/>
-     <joint_properties damping="${ptz_joint_damping}" friction="{ptz_joint_friction}"/>
-  </joint>
-  <transmission name="joint_pan_trans">
-	 <type>transmission_interface/SimpleTransmission</type>
-     <joint name="joint_camera_pan" />
-     <actuator name="pan_motor">
-	   <hardwareInterface>EffortJointInterface</hardwareInterface>
-       <mechanicalReduction>${ptz_mechanical_reduction}</mechanicalReduction>
-     </actuator>
-  </transmission>
-  <link name="camera_tilt_link">
-     <inertial>
-       <mass value="0.1" />
-       <origin xyz="0 0 0" rpy="0 0 0" />
-       <inertia ixx="0.1" ixy="0" ixz="0" iyy="0.1" iyz="0" izz="0.1" />
-    </inertial>
-  </link>
-  <joint name="joint_camera_tilt" type="continuous">
-     <axis xyz="0 1 0" />
-     <origin xyz="0.0 0.0 0.0"/>
-     <parent link="camera_pan_link"/>
-     <child link="camera_tilt_link"/>
-     <limit effort="${ptz_joint_effort_limit}" velocity="${ptz_joint_velocity_limit}" lower="-1.5708" upper="1.5708"/>
-     <joint_properties damping="${ptz_joint_damping}" friction="{ptz_joint_friction}"/>
-  </joint>
-  <transmission name="joint_tilt_trans">
-	 <type>transmission_interface/SimpleTransmission</type>
-     <joint name="joint_camera_tilt" />
-     <actuator name="tilt_motor">
-	   <hardwareInterface>EffortJointInterface</hardwareInterface>
-       <mechanicalReduction>${ptz_mechanical_reduction}</mechanicalReduction>
-     </actuator>
-  </transmission-->
 </robot>
