Commit message: bug fixes collision, joystick
bugs fixed:
# 1768, #1763, #1771

File: guardian_sim/guardian_description/urdf/gball.urdf.xacro (robot description, xacro)
@@ -150,5 +150,5 @@
     </visual>
     <collision>
-       <origin xyz="0 0 0" rpy="0 0 0" />
+       <origin xyz="0 0 0" rpy="0 0 3.1416" />
        <geometry>
          <mesh filename="package://guardian_description/meshes/wheel.dae"/>
@@ -232,5 +232,5 @@
     </visual>
     <collision>
-       <origin xyz="0 0 0" rpy="0 0 0" />
+       <origin xyz="0 0 0" rpy="0 0 3.1416" />
        <geometry>
          <mesh filename="package://guardian_description/meshes/wheel.dae"/>

Commit message: Modified Laser plugin
added plugin libgazebo_ros_laser_2D.so (modified from
libgazebo_ros_laser) which has time_increment, scan_time and option to
not publish intensities[]. Task #1861

changed lasers' names (links, joints...)
front laser is tilt_laser, back laser is base_laser

changed Gazebo laser's specs according to the datasheets
update rate, noise, angles

File: guardian_sim/guardian_description/urdf/gball.urdf.xacro (robot description, xacro)
@@ -313,12 +313,12 @@
   </link>
   <!-- HOKUYO SENSOR -->
-  <joint name="hokuyo_laser_joint" type="fixed">
+  <joint name="hokuyo_base_laser_joint" type="fixed">
      <axis xyz="0 1 0" />
      <origin xyz="0.49 0 0.23"/>
      <parent link="base_link"/>
-     <child link="hokuyo_laser_link"/>
+     <child link="hokuyo_base_laser_link"/>
   </joint>
   <!-- Hokuyo Laser -->
-  <link name="hokuyo_laser_link">
+  <link name="hokuyo_base_laser_link">
     <!-- collision>
       <origin xyz="0 0 0" rpy="0 0 0"/>

File: guardian_sim/guardian_description/urdf/gball_ita.urdf (robot description, URDF)
Before this commit: robot gball, 22 links, 21 joints
Links:
- removed link hokuyo_laser_link
- added link hokuyo_base_laser_link, mass 0.001
Joints:
- removed joint hokuyo_laser_joint
- added joint hokuyo_base_laser_joint: type fixed, parent base_link, child hokuyo_base_laser_link, origin xyz=0.5 0 0.31, axis 0 1 0

File: guardian_sim/guardian_description/urdf/gball_ita_23082013.urdf (robot description, URDF)
Before this commit: robot gball, 22 links, 21 joints
Links:
- removed link hokuyo_laser_link
- added link hokuyo_base_laser_link, mass 0.001
Joints:
- removed joint hokuyo_laser_joint
- added joint hokuyo_base_laser_joint: type fixed, parent base_link, child hokuyo_base_laser_link, origin xyz=0.5 0 0.31, axis 0 1 0

File: guardian_sim/guardian_description/urdf/gball_ita_sinfootprint.urdf (robot description, URDF)
Before this commit: robot gball, 21 links, 20 joints
Links:
- removed link hokuyo_laser_link
- added link hokuyo_base_laser_link, mass 0.001
Joints:
- removed joint hokuyo_laser_joint
- added joint hokuyo_base_laser_joint: type fixed, parent base_link, child hokuyo_base_laser_link, origin xyz=0.5 0 0.31, axis 0 1 0

File: guardian_sim/guardian_description/urdf/guardian.urdf.xacro (robot description, xacro)
@@ -290,29 +290,15 @@
      <!-- motorTorqueConstant>1</motorTorqueConstant -->
   </transmission>
-	<!-- KINECT CAMERA -->
-  <!--joint name="camera_joint" type="fixed">
-     <axis xyz="0 1 0" />
-     <origin xyz="0.5 0 0.31"/>
-     <parent link="base_link"/>
-     <child link="camera_link"/>
-  </joint>
-  <link name="camera_link">
-     <inertial>
-       <mass value="0.001" />
-       <origin xyz="0 0 0" rpy="0 0 0" />
-       <inertia ixx="0.0001" ixy="0" ixz="0" iyy="0.000001" iyz="0" izz="0.0001" />
-    </inertial>
-  </link-->
-  <!-- FRONT - TILT LASER -->
-  <joint name="laser_tilt_joint" type="revolute">
+  <!-- FRONT - TILT LASER - URG-04LX -->
+  <joint name="hokuyo_tilt_laser_joint" type="revolute">
      <axis xyz="0 1 0" />
      <!--origin xyz="0.180 0.0 0.270"/-->
      <origin xyz="0.48856 0 0.24" rpy="0 0 0" /> <!-- 0.1885 --><!--   <origin xyz="0.5 0 0.31" rpy="0 0 0" /> -->
      <parent link="base_link"/>
-     <child link="hokuyo_laser_tilt_link"/>
+     <child link="hokuyo_tilt_laser_link"/>
      <limit effort="${ptz_joint_effort_limit}" velocity="${ptz_joint_velocity_limit}" lower="-1.5708" upper="1.5708"/>
      <joint_properties damping="${ptz_joint_damping}" friction="{ptz_joint_friction}"/>
   </joint>
-  <link name="hokuyo_laser_tilt_link">
+  <link name="hokuyo_tilt_laser_link">
      <inertial>
        <mass value="0.1" />
@@ -335,8 +321,8 @@
       </collision-->
   </link>
-  <transmission name="joint_laser_tilt_trans">
+  <transmission name="joint_tilt_laser_trans">
    <type>transmission_interface/SimpleTransmission</type>
-     <joint name="laser_tilt_joint" />
-     <actuator name="laser_tilt_motor">
+     <joint name="hokuyo_tilt_laser_joint" />
+     <actuator name="tilt_laser_motor">
      <hardwareInterface>EffortJointInterface</hardwareInterface>
        <mechanicalReduction>${ptz_mechanical_reduction}</mechanicalReduction>
@@ -344,12 +330,12 @@
   </transmission>
   <!-- HOKUYO SENSOR -->
-  <joint name="hokuyo_laser_joint" type="fixed">
+  <joint name="hokuyo_base_laser_joint" type="fixed">
      <axis xyz="0 1 0" />
      <origin xyz="-0.43235 0 0.3" rpy="0 0 ${PI}" /> <!--  z: 0.24199 --> <!-- <origin xyz="-0.55 0 0.31" rpy="0 0 ${PI}" /> -->
      <parent link="base_link"/>
-     <child link="hokuyo_laser_link"/>
+     <child link="hokuyo_base_laser_link"/>
   </joint>
   <!-- Hokuyo Laser -->
-  <link name="hokuyo_laser_link">
+  <link name="hokuyo_base_laser_link">
     <!--  collision>
       <origin xyz="0 0 0" rpy="0 0 0"/>

File: guardian_sim/guardian_description/urdf/guardian_ita.urdf (robot description, URDF)
Before this commit: robot gball, 11 links, 10 joints
Links:
- removed link hokuyo_laser_link
- added link hokuyo_base_laser_link, mass 0.001
Joints:
- removed joint hokuyo_laser_joint
- added joint hokuyo_base_laser_joint: type fixed, parent base_link, child hokuyo_base_laser_link, origin xyz=0.5 0 0.31, axis 0 1 0

File: guardian_sim/guardian_description/urdf/gwam_ume.urdf (robot description, URDF)
Before this commit: robot gwam, 18 links, 17 joints
Links:
- removed link hokuyo_laser_link
- added link hokuyo_base_laser_link, mass 0.001
Joints:
- removed joint hokuyo_laser_joint
- added joint hokuyo_base_laser_joint: type fixed, parent base_link, child hokuyo_base_laser_link, origin xyz=0.45 0 0.32, axis 0 1 0

Commit message: Fixed guardian base collision bounding box to avoid front laser beams cutoff. Improved guardian colors and materials to look more like the real platform.

File: guardian_sim/guardian_description/urdf/gball.urdf.xacro (robot description, xacro)
@@ -186,5 +186,5 @@
          <mesh filename="package://guardian_description/meshes/wheel.dae"/>
        </geometry>
-	<material name="gray">
+	<material name="grey">
 		<color rgba="0.3 0.3 0.3 1"/>
       	</material>

File: guardian_sim/guardian_description/urdf/guardian.urdf.xacro (robot description, xacro)
@@ -180,5 +180,5 @@
          <mesh filename="package://guardian_description/meshes/wheel.dae"/>
        </geometry>
-	<material name="gray">
+	<material name="grey">
 		<color rgba="0.3 0.3 0.3 1"/>
       	</material>

File: guardian_sim/guardian_description/urdf/guardian_simple_collision.urdf.xacro (robot description, xacro)
@@ -71,5 +71,6 @@
        <geometry>
 <!--          <mesh filename="package://guardian_description/meshes/chassis/two_lasers/guardian2lasers.dae"/> -->
-		  <box size = "1.127 0.497 0.28"/> <!-- includes tracks, making it just tall enough not to hit the laser beams -->
+		  <!-- <box size = "1.127 0.497 0.28"/> --> <!-- includes tracks, making it just tall enough not to hit the laser beams -->
+		  <box size = "1.127 0.497 0.25"/>
        </geometry>
     </collision>
@@ -300,4 +301,5 @@
      <!--origin xyz="0.180 0.0 0.270"/-->
      <origin xyz="0.48856 0 0.24" rpy="0 0 0" /> <!-- 0.1885 --><!--   <origin xyz="0.5 0 0.31" rpy="0 0 0" /> -->
+     <!-- <origin xyz="0.505 0 0.24" rpy="0 0 0" /> -->
      <parent link="base_link"/>
      <child link="hokuyo_tilt_laser_link"/>

File: guardian_sim/robotnik_powerball_basics/urdf/gball_powerball_robotnik.gazebo.xacro (robot description, xacro)
@@ -20,5 +20,5 @@
 		</gazebo>
 		<gazebo reference="${name}_2_link">
-			<material>Gazebo/Red</material>
+			<material>Gazebo/BlueLaser</material>
 			<gravity>true</gravity>
             <!-- selfCollide>true</selfCollide -->
@@ -30,5 +30,5 @@
 		</gazebo>
 		<gazebo reference="${name}_4_link">
-			<material>Gazebo/Red</material>
+			<material>Gazebo/BlueLaser</material>
 			<gravity>true</gravity>
 			<!-- selfCollide>true</selfCollide -->
@@ -40,5 +40,5 @@
 		</gazebo>
 		<gazebo reference="${name}_6_link">
-			<material>Gazebo/Red</material>
+			<material>Gazebo/BlueLaser</material>
 			<gravity>true</gravity>
             <!-- selfCollide>true</selfCollide -->

File: guardian_sim/robotnik_powerball_basics/urdf/gball_powerball_robotnik.urdf.xacro (robot description, xacro)
@@ -54,6 +54,6 @@
 					<mesh filename="package://robotnik_powerball_basics/meshes/dae/powerball1.dae" />
 				</geometry>
-				<material name="Red">
-					<color rgba="0.5 0.0 0.0 1.0"/>
+				<material name="BlueEmissive">
+					<color rgba="0.3 0.3 0.3 1.0"/>
 				</material>
 			</visual>
@@ -120,6 +120,6 @@
 					<mesh filename="package://robotnik_powerball_basics/meshes/dae/powerball3.dae" />
 				</geometry>
-				<material name="Red">
-					<color rgba="0.5 0.0 0.0 1.0"/>
+				<material name="BlueEmissive">
+					<color rgba="0.3 0.3 0.3 1.0"/>
 				</material>
 			</visual>
@@ -187,6 +187,6 @@
 					<mesh filename="package://robotnik_powerball_basics/meshes/dae/powerball5.dae" />
 				</geometry>
-				<material name="Red">
-					<color rgba="0.5 0.0 0.0 1.0"/>
+				<material name="BlueEmissive">
+					<color rgba="0.3 0.3 0.3 1.0"/>
 				</material>
 			</visual>

Commit message: Changed robot descriptions colors to match those of the real robot.

File: guardian_sim/guardian_description/urdf/gball.urdf.xacro (robot description, xacro)
@@ -49,5 +49,5 @@
      <child link="base_link" />
   </joint>
-  <!-- BASE_LINK (RED) -->
+  <!-- BASE_LINK (DarkGrey) -->
   <link name="base_link">
     <inertial>

File: guardian_sim/guardian_description/urdf/guardian.urdf.xacro (robot description, xacro)
@@ -50,5 +50,5 @@
      <child link="base_link" />
   </joint>
-  <!-- BASE_LINK (RED) -->
+  <!-- BASE_LINK (DarkGrey) -->
   <link name="base_link">
     <inertial>
@@ -317,5 +317,5 @@
           <!--mesh filename="package://guardian_description/meshes/hokuyo-utm30-lx.dae"/>
         </geometry>
-        <material name="Red" />
+        <material name="DarkGrey" />
       </visual-->
       <!-- collision>

File: guardian_sim/guardian_description/urdf/guardian_simple_collision.urdf.xacro (robot description, xacro)
@@ -55,5 +55,5 @@
      <child link="base_link" />
   </joint>
-  <!-- BASE_LINK (RED) -->
+  <!-- BASE_LINK (DarkGrey) -->
   <link name="base_link">
     <inertial>
@@ -67,4 +67,7 @@
 	     <mesh filename="package://guardian_description/meshes/chassis/two_lasers/guardian2lasers.stl"/>
        </geometry>
+		<material name="DarkGrey">
+			<color rgba="0.4 0.4 0.4 1.0" />
+		</material>
     </visual>
     <collision>
@@ -321,5 +324,5 @@
           <!--mesh filename="package://guardian_description/meshes/hokuyo-utm30-lx.dae"/>
         </geometry>
-        <material name="Red" />
+        <material name="DarkGrey" />
       </visual-->
       <!-- collision>

File: guardian_sim/robotnik_powerball_basics/urdf/materials.urdf.xacro (robot description, xacro)
@@ -2,5 +2,6 @@
 <robot>
 	<material name="Red">
-		<color rgba="0.5 0.0 0.0 1.0"/>
+		<color rgba="0.4 0.4 0.4 1.0"/>
+<!-- 		<color rgba="0.5 0.0 0.0 1.0"/> -->
 	</material>
 	<material name="Green">

File: guardian_sim/robotnik_powerball_basics/urdf/powerball_robotnik.gazebo.xacro (robot description, xacro)
@@ -20,5 +20,5 @@
 		</gazebo>
 		<gazebo reference="${name}_2_link">
-			<material>Gazebo/Red</material>
+			<material>Gazebo/DarkGrey</material>
 			<gravity>true</gravity>
             <!-- selfCollide>true</selfCollide -->
@@ -30,5 +30,5 @@
 		</gazebo>
 		<gazebo reference="${name}_4_link">
-			<material>Gazebo/Red</material>
+			<material>Gazebo/DarkGrey</material>
 			<gravity>true</gravity>
 			<!-- selfCollide>true</selfCollide -->
@@ -40,5 +40,5 @@
 		</gazebo>
 		<gazebo reference="${name}_6_link">
-			<material>Gazebo/Red</material>
+			<material>Gazebo/DarkGrey</material>
 			<gravity>true</gravity>
             <!-- selfCollide>true</selfCollide -->

File: guardian_sim/robotnik_powerball_basics/urdf/powerball_robotnik.urdf.xacro (robot description, xacro)
@@ -54,5 +54,5 @@
 					<mesh filename="package://robotnik_powerball_basics/meshes/dae/powerball1.dae" />
 				</geometry>
-				<material name="Red">
+				<material name="DarkGrey">
 					<color rgba="0.5 0.0 0.0 1.0"/>
 				</material>
@@ -120,5 +120,5 @@
 					<mesh filename="package://robotnik_powerball_basics/meshes/dae/powerball3.dae" />
 				</geometry>
-				<material name="Red">
+				<material name="DarkGrey">
 					<color rgba="0.5 0.0 0.0 1.0"/>
 				</material>
@@ -187,5 +187,5 @@
 					<mesh filename="package://robotnik_powerball_basics/meshes/dae/powerball5.dae" />
 				</geometry>
-				<material name="Red">
+				<material name="DarkGrey">
 					<color rgba="0.5 0.0 0.0 1.0"/>
 				</material>
