Commit message: Improved arm xacro.

File: guardian_sim/guardian_description/urdf/schunk_arm.urdf.xacro (robot description, xacro)
@@ -35,14 +35,14 @@
 		<link name="coupler_link">
 			<visual>
-				<origin xyz="0 0 -0.002" rpy="0 0 0" />
-				<geometry>
-					<box size="0.24 0.1 0.002" />
-				</geometry>
+			  <origin xyz="0.02 0 -0.003" rpy="0 0 0" />
+			  <geometry>
+			    <box size="0.29 0.1 0.003" />
+			  </geometry>
 			</visual>
 			<collision>
-				<origin xyz="0 0 -0.002" rpy="0 0 0" />
-				<geometry>
-					<box size="0.24 0.1 0.002" />
-				</geometry>
+			  <origin xyz="0.02 0 -0.003" rpy="0 0 0" />
+			  <geometry>
+			    <box size="0.29 0.1 0.003" />
+			  </geometry>
 			</collision>
 		</link>
@@ -50,46 +50,46 @@
 			<parent link="ft45_link" />
 			<child link="coupler_link" />
-			<origin xyz="0 0 0.002" rpy="0 0 0" />
+			<origin xyz="0 0 0.003" rpy="0 0 0" />
 		</joint>
 		<!-- camera -->
 		<link name="v_camera_link">
-			<visual>
-				<origin xyz="0 0 -0.01" rpy="0 0 0" />
-				<geometry>
-					<box size="0.03 0.07 0.02" />
-				</geometry>
-			</visual>
-			<collision>
-				<origin xyz="0 0 -0.01" rpy="0 0 0" />
-				<geometry>
-					<box size="0.03 0.07 0.02" />
-				</geometry>
-			</collision>
+		  <visual>
+		    <origin xyz="0 0 -0.01" rpy="0 0 0" />
+		    <geometry>
+		      <box size="0.07 0.03 0.02" />
+		    </geometry>
+		  </visual>
+		  <collision>
+		    <origin xyz="0 0 -0.01" rpy="0 0 0" />
+		    <geometry>
+		      <box size="0.07 0.03 0.02" />
+		    </geometry>
+		  </collision>
 		</link>
 		<joint name="v_camera_joint" type="fixed">
 			<parent link="coupler_link" />
 			<child link="v_camera_link" />
-			<origin xyz="-0.095 0 0.02" rpy="0 0 0" />
+			<origin xyz="-0.11 0 0" rpy="0 0 1.5708" />
 		</joint>
 		<!-- projector -->
-		<!-- <link name="projector_link">
-			<visual>
-				<origin xyz="0 0 -0.05" rpy="0 0 0" />
-				<geometry>
-					<box size="0.05 0.15 0.1" />
-				</geometry>
-			</visual>
-			<collision>
-				<origin xyz="0 0 -0.05" rpy="0 0 0" />
-				<geometry>
-					<box size="0.05 0.15 0.1" />
-				</geometry>
-			</collision>
+		<link name="projector_link">
+		  <visual>
+		    <origin xyz="0.05 0 -0.05" rpy="0 0 0" />
+		    <geometry>
+		      <box size="0.155 0.04 0.1" />
+		    </geometry>
+		  </visual>
+		  <collision>
+		    <origin xyz="0.05 0 -0.05" rpy="0 0 0" />
+		    <geometry>
+		      <box size="0.155 0.04 0.1" />
+		    </geometry>
+		  </collision>
 		</link>
 		<joint name="projector_joint" type="fixed">
-			<parent link="coupler_link" />
-			<child link="projector_link" />
-			<origin xyz="0.08 0 0.02" rpy="0 0 0" />
-		</joint> -->
+		  <parent link="coupler_link" />
+		  <child link="projector_link" />
+		  <origin xyz="0.05 -0.075 0.02" rpy="0 0 0" />
+		</joint>
 		<!-- welding tool -->
 		<link name="tool_link">

Commit message: Updated arm xacro.

File: guardian_sim/guardian_description/urdf/schunk_arm.urdf.xacro (robot description, xacro)
@@ -67,9 +67,9 @@
 		  </collision>
 		</link>
-		<joint name="v_camera_joint" type="fixed">
+		<!--joint name="v_camera_joint" type="fixed">
 			<parent link="coupler_link" />
 			<child link="v_camera_link" />
 			<origin xyz="-0.11 0 0" rpy="0 0 1.5708" />
-		</joint>
+		</joint-->
 		<!-- projector -->
 		<link name="projector_link">
@@ -91,4 +91,9 @@
 		  <child link="projector_link" />
 		  <origin xyz="0.05 -0.075 0.02" rpy="0 0 0" />
+		</joint>
+		<joint name="v_camera_joint" type="fixed">
+		  <parent link="projector_link" />
+		  <child link="v_camera_link" />
+		  <origin xyz="-0.227186 0.0744 -0.0052" rpy="0.00322 0.02632 1.56316" />
 		</joint>
 		<!-- welding tool -->
