Commit message: Changed guardian wheels parameterization to allow better in place 360 rotation.
Removed kinect to speedup simulation tests.
Reintroduced imu.

File: guardian_sim/guardian_description/urdf/guardian_base.urdf.xacro (robot description, xacro)
@@ -1,59 +1,57 @@
 <?xml version="1.0"?>
 <robot xmlns:xacro="http://www.ros.org/wiki/xacro">
-  <xacro:include filename="$(find guardian_description)/urdf/guardian_base.gazebo" />
-  <xacro:include filename="$(find guardian_description)/urdf/sensors/kinect.urdf.xacro"/>
-  <xacro:include filename="$(find guardian_description)/urdf/sensors/imu.urdf.xacro"/>
-  <xacro:include filename="$(find guardian_description)/urdf/sensors/hokuyo_front.urdf.xacro"/>
-  <xacro:include filename="$(find guardian_description)/urdf/sensors/hokuyo_back.urdf.xacro"/>
-  <xacro:macro name="guardian_base" params="base_footprint_z">
-	  <!-- BASE FOOTPRINT -->
-	  <!-- base_footprint is a fictitious link(frame) that is on the ground right below base_link origin,
-	             navigation stack depends on this frame -->
-	  <link name="base_footprint">
-	      <visual>
-	          <origin xyz="0 0 0" rpy="0 0 0" />
-	          <geometry>
-	             <box size="0.001 0.001 0.001" />
-	          </geometry>
-	      </visual>
-	  </link>
-	  <joint name="base_footprint_joint" type="fixed">
-	     <!--NB: While you would think this would make it go up, it is oddly reversed.
-	      This moves the joint to 0,0,0 where we want it for rviz, etc. -->
-	<!--      <origin xyz="0 0 0.130" rpy="0 0 0" /> -->
-	<!--      <origin xyz="0 0 0.18" rpy="0 0 0" /> -->
-	     <origin xyz="0 0 ${base_footprint_z}" rpy="0 0 0" />
-	     <parent link="base_footprint"/>
-	     <child link="base_link" />
-	  </joint>
-	  <!-- BASE_LINK (Grey) -->
-	  <link name="base_link">
-	    <inertial>
-	      <mass value="95.0" /> <!-- 95.0 -->
-	      <origin xyz="0 0 0" />
-	      <inertia  ixx="3.737" ixy="0.008"  ixz="-0.144"  iyy="8.311"  iyz="-0.004"  izz="8.893" />
-	    </inertial>
-	    <visual>
-	       <origin xyz="0 0 0" rpy="0 0 0" />
-	       <geometry>
-		     	<mesh filename="package://guardian_description/meshes/chassis/two_lasers/guardian2lasers.stl"/>
-	       </geometry>
-		   <material name="DarkGrey">
-				<color rgba="0.4 0.4 0.4 1.0" />
-			</material>
-	    </visual>
-	    <collision>
-	       <origin xyz="0 0 0.08" rpy="0 0 0 " />
-	       <geometry>
-			  <!-- <box size = "1.127 0.497 0.28"/> --> <!-- includes tracks, making it just tall enough not to hit the laser beams -->
-			  <box size = "1.127 0.497 0.25"/> <!-- this is not enough -->
-	       </geometry>
-	    </collision>
-	  </link>
-	  <!-- ################# SENSORS ################# -->
-  	  <sensor_kinect  parent="base_link"/>
-<!--   	  <sensor_imu  parent="base_link"/> --> <!-- no imu on the platform, so no imu on the simulator -->
-  	  <sensor_hokuyo_front  parent="base_link" prefix="tilt_laser" visualize="false" origin_x="0.48856" origin_z="0.24" origin_yaw="0"/>
-  	  <sensor_hokuyo_back  parent="base_link" prefix="base_laser" visualize="false" origin_x="-0.4323" origin_z="0.3" origin_yaw="${PI}"/>
-  </xacro:macro>
+	<xacro:include filename="$(find guardian_description)/urdf/guardian_base.gazebo" />
+	<!-- <xacro:include filename="$(find guardian_description)/urdf/sensors/kinect.urdf.xacro"/> -->
+	<xacro:include filename="$(find guardian_description)/urdf/sensors/imu.urdf.xacro" />
+	<xacro:include filename="$(find guardian_description)/urdf/sensors/hokuyo_front.urdf.xacro" />
+	<xacro:include filename="$(find guardian_description)/urdf/sensors/hokuyo_back.urdf.xacro" />
+	<xacro:macro name="guardian_base" params="base_footprint_z">
+		<!-- BASE FOOTPRINT -->
+		<!-- base_footprint is a fictitious link(frame) that is on the ground right below base_link origin, navigation stack depends on this frame -->
+		<link name="base_footprint">
+			<visual>
+				<origin xyz="0 0 0" rpy="0 0 0" />
+				<geometry>
+					<box size="0.005 0.005 0.005" />
+				</geometry>
+			</visual>
+		</link>
+		<joint name="base_footprint_joint" type="fixed">
+			<!--NB: While you would think this would make it go up, it is oddly reversed. This moves the joint to 0,0,0 where we want it for rviz, etc. -->
+			<!-- <origin xyz="0 0 0.130" rpy="0 0 0" /> -->
+			<!-- <origin xyz="0 0 0.18" rpy="0 0 0" /> -->
+			<origin xyz="0 0 ${base_footprint_z}" rpy="0 0 0" />
+			<parent link="base_footprint" />
+			<child link="base_link" />
+		</joint>
+		<!-- BASE_LINK (Grey) -->
+		<link name="base_link">
+			<inertial>
+				<mass value="95.0" /> <!-- 95.0 -->
+				<origin xyz="0 0 0" />
+				<inertia ixx="3.737" ixy="0.008" ixz="-0.144" iyy="8.311" iyz="-0.004" izz="8.893" />
+			</inertial>
+			<visual>
+				<origin xyz="0 0 0" rpy="0 0 0" />
+				<geometry>
+					<mesh filename="package://guardian_description/meshes/chassis/two_lasers/guardian2lasers.stl" />
+				</geometry>
+				<material name="DarkGrey">
+					<color rgba="0.4 0.4 0.4 1.0" />
+				</material>
+			</visual>
+			<collision>
+				<origin xyz="0 0 0.08" rpy="0 0 0 " />
+				<geometry>
+					<!-- <box size = "1.127 0.497 0.28"/> --> <!-- includes tracks, making it just tall enough not to hit the laser beams -->
+					<box size="1.127 0.497 0.25" /> <!-- this is not enough -->
+				</geometry>
+			</collision>
+		</link>
+		<!-- ################# SENSORS ################# -->
+		<!-- <sensor_kinect parent="base_link"/> -->
+		<sensor_imu parent="base_link" /> <!-- guardian_robot_control uses imu to update odometry -->
+		<sensor_hokuyo_front parent="base_link" prefix="tilt_laser" visualize="true" origin_x="0.48856" origin_z="0.24" origin_yaw="0" />
+		<sensor_hokuyo_back parent="base_link" prefix="base_laser" visualize="true" origin_x="-0.4323" origin_z="0.3" origin_yaw="${PI}" />
+	</xacro:macro>
 </robot>

File: guardian_sim/guardian_description/urdf/guardian_simple_collision.urdf.xacro (robot description, xacro)
@@ -3,5 +3,5 @@
   <!-- Import all Gazebo-customization elements, including Gazebo colors -->
   <xacro:include filename="$(find guardian_description)/urdf/guardian.gazebo" />
-  <xacro:include filename="$(find guardian_description)/urdf/sensors/kinect.urdf.xacro"/>
+<!--   <xacro:include filename="$(find guardian_description)/urdf/sensors/kinect.urdf.xacro"/> -->
   <!-- Robot mechanical and motor parameters -->
   <xacro:property name="PI" value="3.1415926535897931"/>
@@ -300,5 +300,5 @@
   </transmission>
 <!-- ################# SENSORS ################# -->
-  <sensor_kinect  parent="base_link"/>
+<!--   <sensor_kinect  parent="base_link"/> -->
   <!-- FRONT - TILT LASER - URG-04LX -->
   <joint name="hokuyo_tilt_laser_joint" type="revolute">

File: guardian_sim/guardian_description/urdf/guardian_tracks.urdf.xacro (robot description, xacro)
@@ -5,9 +5,9 @@
 	<xacro:include filename="$(find guardian_description)/urdf/track_wheel.urdf.xacro" />
 	<!-- ###### BASE ###### -->
-	<guardian_base  base_footprint_z="0.069" />
+	<guardian_base base_footprint_z="0.069" />
 	<!-- ###### TRACKS ###### -->
 	<!-- visual -->
 	<track parent="base_link" prefix="left_track" joint_yaw="${PI}" />
-	<track parent="base_link" prefix="right_track" joint_yaw="0"/>
+	<track parent="base_link" prefix="right_track" joint_yaw="0" />
 	<!-- right track collision -->
 	<track_wheel parent="right_track" prefix="right_tw_1" origin_yaw="0" wheel_offset_x="0.3" reflect_y="-1" joint_yaw="0" />
@@ -24,18 +24,20 @@
 	<!-- ###### PLUGIN ###### -->
 	<gazebo> <!-- from hector_gazebo -->
-       <plugin name="diffdrive_plugin_multiwheel" filename="libdiffdrive_plugin_multi_wheel.so">
-          <alwaysOn>true</alwaysOn>
-          <updateRate>10.0</updateRate>
-          <leftJoints>joint_left_tw_1 joint_left_tw_2 joint_left_tw_3 joint_left_tw_4 joint_left_tw_5 </leftJoints>
-          <rightJoints>joint_right_tw_1 joint_right_tw_2 joint_right_tw_3 joint_right_tw_4 joint_right_tw_5 </rightJoints>
-          <wheelSeparation>0.448</wheelSeparation>
-          <wheelDiameter>0.3</wheelDiameter>
-          <torque>20</torque>
-          <robotNamespace>/guardian</robotNamespace>
-          <robotBaseFrame>base_footprint</robotBaseFrame>
-          <commandTopic>cmd_vel</commandTopic>
-          <publishOdometryTf>true</publishOdometryTf>
-          <publishOdometryMsg>true</publishOdometryMsg>
-        </plugin>
-    </gazebo>
+		<plugin name="diffdrive_plugin_multiwheel" filename="libdiffdrive_plugin_multi_wheel.so">
+			<alwaysOn>true</alwaysOn>
+			<updateRate>10.0</updateRate>
+			<leftJoints>joint_left_tw_1 joint_left_tw_2 joint_left_tw_3 joint_left_tw_4 joint_left_tw_5 </leftJoints>
+			<rightJoints>joint_right_tw_1 joint_right_tw_2 joint_right_tw_3 joint_right_tw_4 joint_right_tw_5 </rightJoints>
+			<wheelSeparation>0.448</wheelSeparation>
+			<wheelDiameter>0.3</wheelDiameter>
+			<torque>20</torque>
+			<robotNamespace>/guardian</robotNamespace>
+			<robotBaseFrame>base_footprint</robotBaseFrame>
+			<commandTopic>cmd_vel</commandTopic>
+			<odometryTopic>odom</odometryTopic>
+			<odometryFrame>odom</odometryFrame>
+			<publishOdometryTf>1</publishOdometryTf>
+			<publishOdometryMsg>1</publishOdometryMsg>
+		</plugin>
+	</gazebo>
 </robot>

File: guardian_sim/guardian_description/urdf/guardian_wheels.urdf.xacro (robot description, xacro)
@@ -6,34 +6,35 @@
 	<xacro:include filename="$(find guardian_description)/urdf/track.urdf.xacro" />
 	<xacro:include filename="$(find guardian_description)/urdf/wheel.urdf.xacro" />
-	<!-- ###### BASE ######-->
-	<guardian_base  base_footprint_z="0.18" />
-	<!-- ###### TRACKS ######-->
+	<!-- ###### BASE ###### -->
+	<guardian_base base_footprint_z="0.18" />
+	<!-- ###### TRACKS ###### -->
 	<track parent="base_link" prefix="left_track" joint_yaw="${PI}" />
-	<track parent="base_link" prefix="right_track" joint_yaw="0"/>
+	<track parent="base_link" prefix="right_track" joint_yaw="0" />
 	<!-- track doesn't have collision, but the chassis has a collision bounding box -->
-	<!-- ###### WHEELS ######-->
-	<wheel parent="base_link" prefix="back_left" origin_yaw="${PI}" reflect_link_y="-1" reflect_joint_x="-1" reflect_joint_y="1" />
-	<wheel parent="base_link" prefix="back_right" origin_yaw="0" reflect_link_y="1" reflect_joint_x="-1" reflect_joint_y="-1" />
-	<wheel parent="base_link" prefix="front_left" origin_yaw="${PI}" reflect_link_y="-1" reflect_joint_x="1" reflect_joint_y="1" />
-	<wheel parent="base_link" prefix="front_right" origin_yaw="0" reflect_link_y="1" reflect_joint_x="1" reflect_joint_y="-1" />
-    <!-- ###### WHEELS PLUGINS ######-->
-    <gazebo>
-	    <plugin name="skid_steer_drive_controller" filename="libskid_steer_plugin.so"> <!-- adapted from gazebo_ros_skid_steer_drive -->
-		    <updateRate>100.0</updateRate>
-		    <robotNamespace>/guardian</robotNamespace>
-		    <leftFrontJoint>joint_front_left_wheel</leftFrontJoint>
-		    <rightFrontJoint>joint_front_right_wheel</rightFrontJoint>
-		    <leftRearJoint>joint_back_left_wheel</leftRearJoint>
-		    <rightRearJoint>joint_back_right_wheel</rightRearJoint>
-		    <wheelSeparation>${wheelSeparation}</wheelSeparation>
-		    <wheelDiameter>${wheelDiameter}</wheelDiameter>
-		    <robotBaseFrame>base_footprint</robotBaseFrame>
-		    <torque>70</torque>
-		    <topicName>cmd_vel</topicName> <!-- there is no TopicName element in gazebo_ros_skid_steer_drive plugin   -->
-		    <commandTopic>cmd_vel</commandTopic>
-		    <odometryTopic>odom</odometryTopic> <!-- publishes OdomGazebo because odom is already being published by guardian_robot_pose -->
-		    <odometryFrame>odom</odometryFrame>
-		    <broadcastTF>1</broadcastTF> <!-- defaults to false -->
-	    </plugin>
-  	</gazebo>
+	<!-- ###### WHEELS ###### -->
+	<wheel parent="base_link" prefix="back_left" origin_yaw="${PI}" reflect_link_y="-1" reflect_joint_x="-1" reflect_joint_y="1" material="Gazebo/FlatBlack" />
+	<wheel parent="base_link" prefix="back_right" origin_yaw="0" reflect_link_y="1" reflect_joint_x="-1" reflect_joint_y="-1" material="Gazebo/FlatBlack" />
+	<wheel parent="base_link" prefix="front_left" origin_yaw="${PI}" reflect_link_y="-1" reflect_joint_x="1" reflect_joint_y="1" material="Gazebo/DarkGrey" />
+	<wheel parent="base_link" prefix="front_right" origin_yaw="0" reflect_link_y="1" reflect_joint_x="1" reflect_joint_y="-1" material="Gazebo/DarkGrey" />
+	<!-- ###### WHEELS PLUGINS ###### -->
+	<gazebo>
+		<plugin name="skid_steer_drive_controller" filename="libskid_steer_plugin.so"> <!-- adapted from gazebo_ros_skid_steer_drive -->
+			<updateRate>100.0</updateRate>
+			<robotNamespace>/guardian</robotNamespace>
+			<leftFrontJoint>joint_front_left_wheel</leftFrontJoint>
+			<rightFrontJoint>joint_front_right_wheel</rightFrontJoint>
+			<leftRearJoint>joint_back_left_wheel</leftRearJoint>
+			<rightRearJoint>joint_back_right_wheel</rightRearJoint>
+			<wheelSeparation>${wheelSeparation}</wheelSeparation>
+			<wheelDiameter>${wheelDiameter}</wheelDiameter>
+			<robotBaseFrame>base_footprint</robotBaseFrame>
+			<torque>70</torque> <!-- 20 -->
+			<topicName>cmd_vel</topicName> <!-- there is no TopicName element in gazebo_ros_skid_steer_drive plugin -->
+			<commandTopic>cmd_vel</commandTopic>
+			<odometryTopic>odom_gazebo</odometryTopic> <!-- publishes OdomGazebo because odom is already being published by guardian_robot_pose -->
+			<odometryFrame>odom_gazebo</odometryFrame>
+			<broadcastTF>0</broadcastTF> <!-- defaults to false -->
+			<publishOdometryMsg>0</publishOdometryMsg>
+		</plugin>
+	</gazebo>
 </robot>

File: guardian_sim/guardian_description/urdf/track.urdf.xacro (robot description, xacro)
@@ -1,31 +1,31 @@
 <?xml version="1.0"?>
 <robot xmlns:xacro="http://www.ros.org/wiki/xacro">
-  <xacro:property name="PI" value="3.1415926535897931"/>
-  <xacro:macro name="track" params="parent prefix joint_yaw">
-	  <link name="${prefix}">
+	<xacro:property name="PI" value="3.1415926535897931" />
+	<xacro:macro name="track" params="parent prefix joint_yaw">
+		<link name="${prefix}">
 			<inertial>
-			      <mass value="1.250" />
-			      <origin xyz="0 0 0" />
-			      <inertia  ixx="0.0109375" ixy="0.0"  ixz="0.0"  iyy="0.021125"  iyz="0.0"  izz="0.0109375" /> <!-- original -->
+				<mass value="1.250" />
+				<origin xyz="0 0 0" />
+				<inertia ixx="0.0109375" ixy="0.0" ixz="0.0" iyy="0.021125" iyz="0.0" izz="0.0109375" /> <!-- original -->
 			</inertial>
-		    <visual>
-		        <origin xyz="0 0 0" rpy="0 0 0" />
-		        <geometry>
-			 		<mesh filename="package://guardian_description/meshes/others/v5/trackV5_l.dae"/>
-		        </geometry>
+			<visual>
+				<origin xyz="0 0 0" rpy="0 0 0" />
+				<geometry>
+					<mesh filename="package://guardian_description/meshes/others/v5/trackV5_l.stl" />
+				</geometry>
 				<material name="black">
-		  			<color rgba="0.1 0.1 0.1 1"/>
-		      	</material>
-		    </visual>
-	   </link>
-	  <joint name="joint_${prefix}" type="fixed">
-	    	<parent link="${parent}"/>
-		    <child link="${prefix}"/>
-		    <origin xyz="0.0 0.0 0.0" rpy="0 0 ${joint_yaw}" />
-	  </joint>
-	  <gazebo reference="${prefix}">
-	    <material>Gazebo/DarkGrey</material>
-	    <turnGravityOff>false</turnGravityOff>
-	  </gazebo>
-  </xacro:macro>
+					<color rgba="0.1 0.1 0.1 1" />
+				</material>
+			</visual>
+		</link>
+		<joint name="joint_${prefix}" type="fixed">
+			<parent link="${parent}" />
+			<child link="${prefix}" />
+			<origin xyz="0.0 0.0 0.0" rpy="0 0 ${joint_yaw}" />
+		</joint>
+		<gazebo reference="${prefix}">
+			<material>Gazebo/FlatBlack</material>
+			<turnGravityOff>false</turnGravityOff>
+		</gazebo>
+	</xacro:macro>
 </robot>

File: guardian_sim/guardian_description/urdf/track_wheel.urdf.xacro (robot description, xacro)
@@ -1,73 +1,73 @@
 <?xml version="1.0"?>
 <robot xmlns:xacro="http://www.ros.org/wiki/xacro">
-  <xacro:property name="PI" value="3.1415926535897931"/>
-  <xacro:property name="mass" value="0.25" />
-   <xacro:property name="simple_wheel_length" value="0.05" />
-  <xacro:property name="simple_wheel_radius" value="0.15" />
-<!--   <xacro:property name="wheel_origin_y" value="0.0" /> -->
-  <xacro:property name="wheel_offset_y" value="0.224" />
-  <xacro:property name="wheel_offset_z" value="0.081" /> <!-- 0.15-0.069 -->
-  <xacro:property name="wheel_joint_damping" value="0.0" />
-  <xacro:property name="wheel_joint_friction" value="0.0" />
-  <xacro:property name="wheel_joint_effort_limit" value="200.0" />
-  <xacro:property name="wheel_joint_velocity_limit" value="200.0" />
-  <xacro:property name="wheel_mechanical_reduction" value="1.0" />
-  <xacro:macro name="track_wheel" params="parent prefix origin_yaw wheel_offset_x reflect_y joint_yaw">
-	  <link name="${prefix}">
-		<inertial>
-		    <mass value="${mass}" /> <!-- 4.5 -->
-		    <origin xyz="0 0 0" rpy="0 0 ${origin_yaw}" />
-		    <inertia  ixx="0.059" ixy="0.0"  ixz="0.0"  iyy="0.055"  iyz="0.0"  izz="0.059" />
-<!-- 			  <inertia  ixx="0.00012411765597" ixy="0.0" ixz="0.0" -->
-<!--                         iyy="0.00015218160428" iyz="0.0" -->
-<!--                         izz="0.00011763977943" /> -->
-<!-- 				  <inertia  ixx="${(1/12)*mass*(3*simple_wheel_radius * simple_wheel_radius + simple_wheel_length*simple_wheel_length)}" ixy="0.0"  ixz="0.0"   -->
-<!-- 		      			    iyy="${(1/12)*mass*(3*simple_wheel_radius * simple_wheel_radius + simple_wheel_length*simple_wheel_length)}" iyz="0.0"   -->
-<!-- 		      			    izz="${0.5*mass*(simple_wheel_radius * simple_wheel_radius)}" />   wikipedia formula -->
-		</inertial>
-<!-- 	    <visual> -->
-<!-- 	        <origin xyz="0 ${reflect_y * wheel_origin_y} 0" rpy="${PI/2} 0 ${origin_yaw}" /> -->
-<!-- 	        <geometry> -->
-<!-- 		 		 <cylinder length="${simple_wheel_length}" radius="${simple_wheel_radius}"/> -->
-<!-- 	        </geometry> -->
-<!-- 			<material name="black"> -->
-<!-- 	  			<color rgba="0.1 0.1 0.1 1"/> -->
-<!-- 	      	</material> -->
-<!-- 	    </visual>	     -->
-		<collision>
-	       <origin xyz="0 0 0" rpy="${PI/2} 0 ${origin_yaw}" />
-	       <geometry>
-	          <cylinder length="${simple_wheel_length}" radius="${simple_wheel_radius}"/>
-	       </geometry>
-<!-- 	       <material name="black"/> -->
-	    </collision>
-	  </link>
-	  <joint name="joint_${prefix}" type="continuous">
-	    	<parent link="${parent}"/>
-		    <child link="${prefix}"/>
-		 	<origin xyz="${wheel_offset_x} ${reflect_y * wheel_offset_y} ${wheel_offset_z}" rpy="0 0 ${joint_yaw}" />
-		    <axis xyz="0 1 0" rpy="0 0 0" />
-		    <limit effort="${wheel_joint_effort_limit}" velocity="${wheel_joint_velocity_limit}"/>
-		    <joint_properties damping="${wheel_joint_damping}" friction="{wheel_joint_friction}"/>
-	  </joint>
-	 <transmission name="joint_${prefix}_trans">
-		 <type>transmission_interface/SimpleTransmission</type>
-	     <joint name="joint_${prefix}" />
-	     <actuator name="joint_${prefix}_motor">
-		    <hardwareInterface>EffortJointInterface</hardwareInterface>
-			<!-- hardwareInterface>VelocityJointInterface</hardwareInterface -->
-	        <mechanicalReduction>${wheel_mechanical_reduction}</mechanicalReduction>
-	     	<!-- motorTorqueConstant>1</motorTorqueConstant -->
-	     </actuator>
-  	 </transmission>
-	 <gazebo reference="${prefix}">
-<!-- 	    <material>Gazebo/Grey</material> -->
-	    <turnGravityOff>false</turnGravityOff>
-		<mu1 value="3"/>
-	    <mu2 value="0.9"/>
-	    <fdir1 value="1 0 0"/>
-	   	<kp value="10000000.0" />
-		<kd value="10.0"/>
-	 </gazebo>
-  </xacro:macro>
+	<xacro:property name="PI" value="3.1415926535897931" />
+	<xacro:property name="mass" value="0.25" />
+	<xacro:property name="simple_wheel_length" value="0.05" />
+	<xacro:property name="simple_wheel_radius" value="0.15" />
+	<!-- <xacro:property name="wheel_origin_y" value="0.0" /> -->
+	<xacro:property name="wheel_offset_y" value="0.224" />
+	<xacro:property name="wheel_offset_z" value="0.081" /> <!-- 0.15-0.069 -->
+	<xacro:property name="wheel_joint_damping" value="0.0" />
+	<xacro:property name="wheel_joint_friction" value="0.0" />
+	<xacro:property name="wheel_joint_effort_limit" value="200.0" />
+	<xacro:property name="wheel_joint_velocity_limit" value="200.0" />
+	<xacro:property name="wheel_mechanical_reduction" value="1.0" />
+	<xacro:macro name="track_wheel" params="parent prefix origin_yaw wheel_offset_x reflect_y joint_yaw">
+		<link name="${prefix}">
+			<inertial>
+				<mass value="${mass}" /> <!-- 4.5 -->
+				<origin xyz="0 0 0" rpy="0 0 ${origin_yaw}" />
+				<inertia ixx="0.059" ixy="0.0" ixz="0.0" iyy="0.055" iyz="0.0" izz="0.059" />
+				<!-- <inertia ixx="0.00012411765597" ixy="0.0" ixz="0.0" -->
+				<!-- iyy="0.00015218160428" iyz="0.0" -->
+				<!-- izz="0.00011763977943" /> -->
+				<!-- <inertia ixx="${(1/12)*mass*(3*simple_wheel_radius * simple_wheel_radius + simple_wheel_length*simple_wheel_length)}" ixy="0.0" ixz="0.0" -->
+				<!-- iyy="${(1/12)*mass*(3*simple_wheel_radius * simple_wheel_radius + simple_wheel_length*simple_wheel_length)}" iyz="0.0" -->
+				<!-- izz="${0.5*mass*(simple_wheel_radius * simple_wheel_radius)}" /> wikipedia formula -->
+			</inertial>
+			<!-- <visual> -->
+			<!-- <origin xyz="0 ${reflect_y * wheel_origin_y} 0" rpy="${PI/2} 0 ${origin_yaw}" /> -->
+			<!-- <geometry> -->
+			<!-- <cylinder length="${simple_wheel_length}" radius="${simple_wheel_radius}"/> -->
+			<!-- </geometry> -->
+			<!-- <material name="black"> -->
+			<!-- <color rgba="0.1 0.1 0.1 1"/> -->
+			<!-- </material> -->
+			<!-- </visual> -->
+			<collision>
+				<origin xyz="0 0 0" rpy="${PI/2} 0 ${origin_yaw}" />
+				<geometry>
+					<cylinder length="${simple_wheel_length}" radius="${simple_wheel_radius}" />
+				</geometry>
+				<!-- <material name="black"/> -->
+			</collision>
+		</link>
+		<joint name="joint_${prefix}" type="continuous">
+			<parent link="${parent}" />
+			<child link="${prefix}" />
+			<origin xyz="${wheel_offset_x} ${reflect_y * wheel_offset_y} ${wheel_offset_z}" rpy="0 0 ${joint_yaw}" />
+			<axis xyz="0 1 0" rpy="0 0 0" />
+			<limit effort="${wheel_joint_effort_limit}" velocity="${wheel_joint_velocity_limit}" />
+			<joint_properties damping="${wheel_joint_damping}" friction="{wheel_joint_friction}" />
+		</joint>
+		<transmission name="joint_${prefix}_trans">
+			<type>transmission_interface/SimpleTransmission</type>
+			<joint name="joint_${prefix}" />
+			<actuator name="joint_${prefix}_motor">
+				<hardwareInterface>EffortJointInterface</hardwareInterface>
+				<!-- hardwareInterface>VelocityJointInterface</hardwareInterface -->
+				<mechanicalReduction>${wheel_mechanical_reduction}</mechanicalReduction>
+				<!-- motorTorqueConstant>1</motorTorqueConstant -->
+			</actuator>
+		</transmission>
+		<gazebo reference="${prefix}">
+			<!-- <material>Gazebo/Grey</material> -->
+			<turnGravityOff>false</turnGravityOff>
+			<mu1 value="3" />
+			<mu2 value="0.9" />
+			<fdir1 value="1 0 0" />
+			<kp value="10000000.0" />
+			<kd value="10.0" />
+		</gazebo>
+	</xacro:macro>
 </robot>
