Commit message: Changed guardian wheels parameterization to allow better in place 360 rotation.
Removed kinect to speedup simulation tests.
Reintroduced imu.

File: guardian_sim/guardian_description/urdf/wheel.urdf.xacro (robot description, xacro)
@@ -1,70 +1,71 @@
 <?xml version="1.0"?>
 <robot xmlns:xacro="http://www.ros.org/wiki/xacro">
-  <xacro:property name="PI" value="3.1415926535897931"/>
-  <xacro:property name="mass" value="4.3"/>
-  <xacro:property name="simple_wheel_length" value="0.115" />
-  <xacro:property name="simple_wheel_radius" value="0.185" />
-  <xacro:property name="wheel_origin_y" value="0.03" />
-  <xacro:property name="wheel_offset_x" value="0.300" />
-  <xacro:property name="wheel_offset_y" value="0.306" />
-  <xacro:property name="wheel_joint_damping" value="0.0" />
-  <xacro:property name="wheel_joint_friction" value="0.0" />
-  <xacro:property name="wheel_joint_effort_limit" value="200.0" />
-  <xacro:property name="wheel_joint_velocity_limit" value="200.0" />
-  <xacro:property name="wheel_mechanical_reduction" value="1.0" />
-  <xacro:macro name="wheel" params="parent prefix origin_yaw reflect_link_y reflect_joint_x reflect_joint_y">
-	  <link name="${prefix}_wheel">
-		    <inertial>
-		       <mass value="${mass}" />
-		       <origin xyz="0 0 0" rpy="0 0 ${origin_yaw}" />
-<!-- 		      <inertia  ixx="0.059" ixy="0.0"  ixz="0.0"  iyy="0.055"  iyz="0.0"  izz="0.059" />  original (robotnik)    -->
-		       <inertia  ixx="${(1/12)*mass*(3*simple_wheel_radius * simple_wheel_radius + simple_wheel_length*simple_wheel_length)}" ixy="0.0"  ixz="0.0"
-		      			 iyy="${(1/12)*mass*(3*simple_wheel_radius * simple_wheel_radius + simple_wheel_length*simple_wheel_length)}" iyz="0.0"
-		      			 izz="${0.5*mass*(simple_wheel_radius * simple_wheel_radius)}" />
-		    </inertial>
-	    <visual> <!-- visual wheels need offset because their origin is not in the center of the wheel -->
-	        <origin xyz="0 ${reflect_link_y * wheel_origin_y} 0" rpy="0 0 ${origin_yaw}" />
-	        <geometry>
-		 		<mesh filename="package://guardian_description/meshes/wheel.stl"/>
-	        </geometry>
-			<material name="black">
-	  			<color rgba="0.1 0.1 0.1 1"/>
-	      	</material>
-	    </visual>
-		<collision>
-	       <origin xyz="0 0 0" rpy="${PI/2} 0 0" />
-	       <geometry>
-	          <cylinder length="${simple_wheel_length}" radius="${simple_wheel_radius}"/>
-	       </geometry>
-	       <material name="black"/>
-	    </collision>
-	  </link>
-	  <joint name="joint_${prefix}_wheel" type="continuous">
-	    	<parent link="${parent}"/>
-		    <child link="${prefix}_wheel"/>
-		 	  <origin xyz="${reflect_joint_x * wheel_offset_x} ${reflect_joint_y * wheel_offset_y} 0" rpy="0 0 0" />
-		    <axis xyz="0 1 0" rpy="0 0 0" />
-		    <limit effort="${wheel_joint_effort_limit}" velocity="${wheel_joint_velocity_limit}"/>
-		    <joint_properties damping="${wheel_joint_damping}" friction="{wheel_joint_friction}"/>
-	  </joint>
-	 <transmission name="joint_${prefix}_trans">
-		 <type>transmission_interface/SimpleTransmission</type>
-	     <joint name="joint_${prefix}_wheel" />
-	     <actuator name="joint_${prefix}_motor">
-		    <hardwareInterface>EffortJointInterface</hardwareInterface>
-			<!-- hardwareInterface>VelocityJointInterface</hardwareInterface -->
-	        <mechanicalReduction>${wheel_mechanical_reduction}</mechanicalReduction>
-	     	<!-- motorTorqueConstant>1</motorTorqueConstant -->
-	     </actuator>
-  	 </transmission>
-	 <gazebo reference="${prefix}_wheel">
-	    <material>Gazebo/DarkGrey</material>
-	    <turnGravityOff>false</turnGravityOff>
-		<mu1 value="3"/>
-	    <mu2 value="0.9"/>
-	    <fdir1 value="1 0 0"/>
-	   	<kp value="10000000.0" />
-		<kd value="10.0"/>
-	 </gazebo>
-  </xacro:macro>
+	<xacro:property name="PI" value="3.1415926535897931" />
+	<xacro:property name="mass" value="4.3" />
+	<xacro:property name="simple_wheel_length" value="0.1143" />
+	<xacro:property name="simple_wheel_radius" value="0.1850" />
+	<xacro:property name="wheel_origin_y" value="0.03" />
+	<xacro:property name="wheel_offset_x" value="0.300" />
+	<xacro:property name="wheel_offset_y" value="0.306" />
+	<xacro:property name="wheel_joint_damping" value="0.0" />
+	<xacro:property name="wheel_joint_friction" value="0.0" />
+	<xacro:property name="wheel_joint_effort_limit" value="200.0" />
+	<xacro:property name="wheel_joint_velocity_limit" value="200.0" />
+	<xacro:property name="wheel_mechanical_reduction" value="1.0" />
+	<xacro:macro name="wheel" params="parent prefix origin_yaw reflect_link_y reflect_joint_x reflect_joint_y material">
+		<link name="${prefix}_wheel">
+			<inertial>
+				<mass value="${mass}" />
+				<origin xyz="0 0 0" rpy="0 0 ${origin_yaw}" />
+				<!-- <inertia ixx="0.059" ixy="0.0" ixz="0.0" iyy="0.055" iyz="0.0" izz="0.059" /> original (robotnik) -->
+				<inertia ixx="${(1/12)*mass*(3*simple_wheel_radius * simple_wheel_radius + simple_wheel_length*simple_wheel_length)}" ixy="0.0" ixz="0.0"
+					iyy="${(1/12)*mass*(3*simple_wheel_radius * simple_wheel_radius + simple_wheel_length*simple_wheel_length)}" iyz="0.0" izz="${0.5*mass*(simple_wheel_radius * simple_wheel_radius)}" />
+			</inertial>
+			<visual> <!-- visual wheels need offset because their origin is not in the center of the wheel -->
+				<origin xyz="0 ${reflect_link_y * wheel_origin_y} 0" rpy="0 0 ${origin_yaw}" />
+				<geometry>
+					<mesh filename="package://guardian_description/meshes/wheel.stl" />
+				</geometry>
+			</visual>
+			<collision>
+				<origin xyz="0 ${reflect_link_y * -0.012} 0" rpy="${PI/2} 0 0" /> <geometry> <cylinder length="${simple_wheel_length}" radius="${simple_wheel_radius}"/> </geometry>
+<!-- 				<origin xyz="0 ${reflect_link_y * wheel_origin_y} 0" rpy="0 0 ${origin_yaw}" /> <geometry> <mesh filename="package://guardian_description/meshes/wheel.stl" /> </geometry> -->
+			</collision>
+		</link>
+		<joint name="joint_${prefix}_wheel" type="continuous">
+			<parent link="${parent}" />
+			<child link="${prefix}_wheel" />
+			<origin xyz="${reflect_joint_x * wheel_offset_x} ${reflect_joint_y * wheel_offset_y} 0" rpy="0 0 0" />
+			<axis xyz="0 1 0" rpy="0 0 0" />
+			<limit effort="${wheel_joint_effort_limit}" velocity="${wheel_joint_velocity_limit}" />
+			<joint_properties damping="${wheel_joint_damping}" friction="{wheel_joint_friction}" />
+		</joint>
+		<transmission name="joint_${prefix}_trans">
+			<type>transmission_interface/SimpleTransmission</type>
+			<joint name="joint_${prefix}_wheel" />
+			<actuator name="joint_${prefix}_motor">
+				<hardwareInterface>EffortJointInterface</hardwareInterface>
+				<!-- hardwareInterface>VelocityJointInterface</hardwareInterface -->
+				<mechanicalReduction>${wheel_mechanical_reduction}</mechanicalReduction>
+				<!-- motorTorqueConstant>1</motorTorqueConstant -->
+			</actuator>
+		</transmission>
+		<gazebo reference="${prefix}_wheel">
+			<material>${material}</material>
+			<turnGravityOff>false</turnGravityOff>
+			<fdir1 value="1 0 0" /> <!-- direction of mu1 -->
+			<maxVel>2.0</maxVel>
+			<maxContacts>3</maxContacts>
+			<minDepth>0.0025</minDepth>
+			<mu1 value="0.55" /> <!-- [0..1] | friction coefficient x -->
+			<mu2 value="0.35" /> <!-- [0..1] | friction coefficient y -->
+			<kp value="95000" /> <!-- stiffness -->
+			<kd value="300" /> <!-- damping -->
+			<!-- <mu1 value="0.55" />
+			<mu2 value="0.35" />
+			<kp value="95000.0" />
+			<kd value="300.0" /> -->
+			<maxVel>2.0</maxVel>
+		</gazebo>
+	</xacro:macro>
 </robot>

Commit message: Uniformization of topic names and namespaces.

File: guardian_sim/guardian_description/urdf/guardian_base.urdf.xacro (robot description, xacro)
@@ -2,5 +2,5 @@
 <robot xmlns:xacro="http://www.ros.org/wiki/xacro">
 	<xacro:include filename="$(find guardian_description)/urdf/guardian_base.gazebo" />
-	<!-- <xacro:include filename="$(find guardian_description)/urdf/sensors/kinect.urdf.xacro"/> -->
+	<xacro:include filename="$(find guardian_description)/urdf/sensors/kinect.urdf.xacro"/>
 	<xacro:include filename="$(find guardian_description)/urdf/sensors/imu.urdf.xacro" />
 	<xacro:include filename="$(find guardian_description)/urdf/sensors/hokuyo_front.urdf.xacro" />
@@ -50,5 +50,5 @@
 		</link>
 		<!-- ################# SENSORS ################# -->
-		<!-- <sensor_kinect parent="base_link"/> -->
+		<sensor_kinect parent="base_link"/>
 		<sensor_imu parent="base_link" /> <!-- guardian_robot_control uses imu to update odometry -->
 		<sensor_hokuyo_front parent="base_link" prefix="tilt_laser" visualize="true" origin_x="0.48856" origin_z="0.24" origin_yaw="0" />

File: guardian_sim/guardian_description/urdf/guardian_wheels.urdf.xacro (robot description, xacro)
@@ -29,5 +29,5 @@
 			<wheelDiameter>${wheelDiameter}</wheelDiameter>
 			<robotBaseFrame>base_footprint</robotBaseFrame>
-			<torque>70</torque> <!-- 20 -->
+			<torque>200</torque> <!-- 20 -->
 			<topicName>cmd_vel</topicName> <!-- there is no TopicName element in gazebo_ros_skid_steer_drive plugin -->
 			<commandTopic>cmd_vel</commandTopic>

File: guardian_sim/guardian_description/urdf/sensors/hokuyo_back.urdf.xacro (robot description, xacro)
@@ -1,73 +1,64 @@
 <?xml version="1.0"?>
 <robot xmlns:xacro="http://www.ros.org/wiki/xacro">
-  <!-- Robot parameters -->
-  <xacro:property name="PI" value="3.1415926535897931"/>
-  <xacro:property name="ptz_joint_effort_limit" value="100.0" />
-  <xacro:property name="ptz_joint_velocity_limit" value="100.0"/>
-  <xacro:property name="ptz_joint_friction" value="0.1" />
-  <xacro:property name="ptz_joint_damping" value="0.1" />
-  <xacro:property name="ptz_mechanical_reduction" value="1.0" />
-  <xacro:macro name="sensor_hokuyo_back" params="parent prefix visualize origin_x origin_z origin_yaw">
- 	<!-- joint -->
-	  <joint name="hokuyo_${prefix}_joint" type="fixed">
-	     <axis xyz="0 1 0" />
-	     <origin xyz="${origin_x} 0 ${origin_z}" rpy="0 0 ${origin_yaw}" />
-	     <parent link="${parent}"/>
-	     <child link="hokuyo_${prefix}_link"/>
-	  </joint>
- 	<!-- link -->
-	  <link name="hokuyo_${prefix}_link">
-	     <inertial>
-	       <mass value="0.1" />
-	       <origin xyz="0 0 0" rpy="0 0 0" />
-	       <inertia ixx="0.1" ixy="0" ixz="0" iyy="0.1" iyz="0" izz="0.1" />
-	    </inertial>
-<!--
-		<inertial>
-	       <mass value="1e-5" />
-     	   <origin xyz="0 0 0" rpy="0 0 0"/>
-      	   <inertia ixx="1e-6" ixy="0" ixz="0" iyy="1e-6" iyz="0" izz="1e-6" />
-    	</inertial>
--->
-	  </link>
-	<!-- gazebo -->
-	  <gazebo reference="hokuyo_${prefix}_link">
-	    <material>Gazebo/FlatBlack</material>
-	    <sensor type="ray" name="${prefix}_sensor">
-	      <pose>0 0 0 0 0 0</pose>
-	      <visualize>${visualize}</visualize>
-	      <update_rate>10</update_rate> <!-- rate of 10 for scan time ~ 100 ms  -->
-	      <ray>
-	        <scan>
-	          <horizontal>
-	           <samples>684</samples> <!-- 683 steps + 1 -->
-	           <resolution>1</resolution>
-	           <min_angle>-2.0943951</min_angle>  <!-- 120+120 deg in the back-->
-	           <max_angle>2.0943951</max_angle>
-	          </horizontal>
-	        </scan>
-	        <range>
-	          <min>0.10</min>
-	          <max>5.0</max> <!-- 5.0 -->
-	          <resolution>0.001</resolution> <!-- 0.001 -->
-	        </range>
-	        <noise>
-	          <type>gaussian</type>
-	          <!-- Noise parameters based on published spec for Hokuyo laser
-	               achieving "+-30mm" accuracy at range < 10m.  A mean of 0.0m and
-	               stddev of 0.01m will put 99.7% of samples within 0.03m of the true
-	               reading. -->
-	          <mean>0.0</mean>
-	          <stddev>0.01</stddev> <!-- 0.01 -->
-	        </noise>
-	      </ray>
-	      <plugin name="${prefix}_plugin" filename="libgazebo_ros_laser_2D.so">
-	        <topicName>/back_horizontal_scan</topicName>
-	        <frameName>hokuyo_${prefix}_link</frameName>
-	        <time_increment>0.00009765739</time_increment> <!-- time between measurements --> <!-- 0.0667 sec /683 steps -->
-	        <intensities>0</intensities> <!-- Whether or not the hokuyo laser returns intensity values. 0 means no intensities[] -->
-	      </plugin>
-	    </sensor>
-	  </gazebo>
-  </xacro:macro>
+	<!-- Robot parameters -->
+	<xacro:property name="PI" value="3.1415926535897931" />
+	<xacro:property name="ptz_joint_effort_limit" value="100.0" />
+	<xacro:property name="ptz_joint_velocity_limit" value="100.0" />
+	<xacro:property name="ptz_joint_friction" value="0.1" />
+	<xacro:property name="ptz_joint_damping" value="0.1" />
+	<xacro:property name="ptz_mechanical_reduction" value="1.0" />
+	<xacro:macro name="sensor_hokuyo_back" params="parent prefix visualize origin_x origin_z origin_yaw">
+		<!-- joint -->
+		<joint name="hokuyo_${prefix}_joint" type="fixed">
+			<axis xyz="0 1 0" />
+			<origin xyz="${origin_x} 0 ${origin_z}" rpy="0 0 ${origin_yaw}" />
+			<parent link="${parent}" />
+			<child link="hokuyo_${prefix}_link" />
+		</joint>
+		<!-- link -->
+		<link name="hokuyo_${prefix}_link">
+			<inertial>
+				<mass value="0.1" />
+				<origin xyz="0 0 0" rpy="0 0 0" />
+				<inertia ixx="0.1" ixy="0" ixz="0" iyy="0.1" iyz="0" izz="0.1" />
+			</inertial>
+			<!-- <inertial> <mass value="1e-5" /> <origin xyz="0 0 0" rpy="0 0 0"/> <inertia ixx="1e-6" ixy="0" ixz="0" iyy="1e-6" iyz="0" izz="1e-6" /> </inertial> -->
+		</link>
+		<!-- gazebo -->
+		<gazebo reference="hokuyo_${prefix}_link">
+			<material>Gazebo/FlatBlack</material>
+			<sensor type="ray" name="${prefix}_sensor">
+				<pose>0 0 0 0 0 0</pose>
+				<visualize>${visualize}</visualize>
+				<update_rate>10</update_rate> <!-- rate of 10 for scan time ~ 100 ms -->
+				<ray>
+					<scan>
+						<horizontal>
+							<samples>684</samples> <!-- 683 steps + 1 -->
+							<resolution>1</resolution>
+							<min_angle>-2.0943951</min_angle>  <!-- 120+120 deg in the back -->
+							<max_angle>2.0943951</max_angle>
+						</horizontal>
+					</scan>
+					<range>
+						<min>0.10</min>
+						<max>5.0</max> <!-- 5.0 -->
+						<resolution>0.001</resolution> <!-- 0.001 -->
+					</range>
+					<noise>
+						<type>gaussian</type>
+						<!-- Noise parameters based on published spec for Hokuyo laser achieving "+-30mm" accuracy at range < 10m. A mean of 0.0m and stddev of 0.01m will put 99.7% of samples within 0.03m of the true reading. -->
+						<mean>0.0</mean>
+						<stddev>0.01</stddev> <!-- 0.01 -->
+					</noise>
+				</ray>
+				<plugin name="${prefix}_plugin" filename="libgazebo_ros_laser_2D.so">
+					<topicName>/guardian/laser_horizontal_back</topicName>
+					<frameName>hokuyo_${prefix}_link</frameName>
+					<time_increment>0.00009765739</time_increment> <!-- time between measurements --> <!-- 0.0667 sec /683 steps -->
+					<intensities>0</intensities> <!-- Whether or not the hokuyo laser returns intensity values. 0 means no intensities[] -->
+				</plugin>
+			</sensor>
+		</gazebo>
+	</xacro:macro>
 </robot>

File: guardian_sim/guardian_description/urdf/sensors/hokuyo_front.urdf.xacro (robot description, xacro)
@@ -64,5 +64,5 @@
 	      </ray>
 	      <plugin name="${prefix}_plugin" filename="libgazebo_ros_laser_2D.so">
-	        <topicName>/front_tilt_scan</topicName>
+	        <topicName>/guardian/laser_tilt_front</topicName>
 	        <frameName>hokuyo_${prefix}_link</frameName>
 	        <time_increment>0.00009765739</time_increment> <!-- time between measurements --> <!-- 0.0667 sec /683 steps -->

File: guardian_sim/guardian_description/urdf/sensors/kinect_gazebo.urdf.xacro (robot description, xacro)
@@ -6,7 +6,7 @@
       <sensor type="depth" name="camera">
         <always_on>true</always_on>
-        <update_rate>30.0</update_rate>
+        <update_rate>30.0</update_rate> <!-- specs -> 30 -->
         <camera>
-          <horizontal_fov>${57.0*M_PI/180.0}</horizontal_fov>
+          <horizontal_fov>${43*M_PI/180.0}</horizontal_fov> <!-- specs: 43.0*M_PI/180.0 -->
           <!-- <vertical_fov>${43.0*M_PI/180.0}</vertical_fov> -->
           <image>
@@ -16,6 +16,6 @@
           </image>
           <clip>
-            <near>0.8</near>
-            <far>4.0</far>
+            <near>0.8</near> <!-- specs -> 0.8 -->
+            <far>4.0</far> <!-- specs -> 4.0 -->
           </clip>
         </camera>
@@ -23,5 +23,5 @@
           <cameraName>camera</cameraName>
           <alwaysOn>true</alwaysOn>
-          <updateRate>30</updateRate>
+          <updateRate>30.0</updateRate> <!-- specs -> 30 -->
           <imageTopicName>rgb/image_raw</imageTopicName>
           <depthImageTopicName>depth/image_raw</depthImageTopicName>
@@ -36,5 +36,5 @@
           <distortion_t1>0.0</distortion_t1>
           <distortion_t2>0.0</distortion_t2>
-          <pointCloudCutoff>0.8</pointCloudCutoff>
+          <pointCloudCutoff>0.8</pointCloudCutoff> <!-- specs -> 0.8 -->
         </plugin>
       </sensor>

File: guardian_sim/guardian_description/urdf/wheel.urdf.xacro (robot description, xacro)
@@ -54,17 +54,16 @@
 			<material>${material}</material>
 			<turnGravityOff>false</turnGravityOff>
-			<fdir1 value="1 0 0" /> <!-- direction of mu1 -->
-			<maxVel>2.0</maxVel>
-			<maxContacts>3</maxContacts>
+			<!-- <fdir1 value="1 0 0" /> --> <!-- direction of mu1 -->
+			<maxContacts>6</maxContacts>
 			<minDepth>0.0025</minDepth>
-			<mu1 value="0.55" /> <!-- [0..1] | friction coefficient x -->
-			<mu2 value="0.35" /> <!-- [0..1] | friction coefficient y -->
-			<kp value="95000" /> <!-- stiffness -->
-			<kd value="300" /> <!-- damping -->
+			<mu1 value="0.85" /> <!-- [0..1] | friction coefficient x -->
+			<mu2 value="0.75" /> <!-- [0..1] | friction coefficient y -->
+			<kp value="55000" /> <!-- stiffness -->
+			<kd value="350" /> <!-- damping -->
 			<!-- <mu1 value="0.55" />
 			<mu2 value="0.35" />
 			<kp value="95000.0" />
 			<kd value="300.0" /> -->
-			<maxVel>2.0</maxVel>
+			<!-- <maxVel>2.0</maxVel> -->
 		</gazebo>
 	</xacro:macro>

Commit message: Updated front laser URDF to the current (elevated) position

File: guardian_sim/guardian_description/urdf/guardian_base.urdf.xacro (robot description, xacro)
@@ -52,5 +52,5 @@
 		<sensor_kinect parent="base_link"/>
 		<sensor_imu parent="base_link" /> <!-- guardian_robot_control uses imu to update odometry -->
-		<sensor_hokuyo_front parent="base_link" prefix="tilt_laser" visualize="true" origin_x="0.48856" origin_z="0.24" origin_yaw="0" />
+		<sensor_hokuyo_front parent="base_link" prefix="tilt_laser" visualize="true" origin_x="0.46781" origin_z="0.24299" origin_yaw="0" />
 		<sensor_hokuyo_back parent="base_link" prefix="base_laser" visualize="true" origin_x="-0.4323" origin_z="0.3" origin_yaw="${PI}" />
 	</xacro:macro>

File: guardian_sim/guardian_description/urdf/sensors/hokuyo_front.urdf.xacro (robot description, xacro)
@@ -8,34 +8,65 @@
   <xacro:property name="ptz_joint_damping" value="0.1" />
   <xacro:property name="ptz_mechanical_reduction" value="1.0" />
+  <xacro:property name="laser_offset_z" value="0.06" />
   <xacro:macro name="sensor_hokuyo_front" params="parent prefix visualize origin_x origin_z origin_yaw">
- 	<!-- joint -->
-	  <joint name="hokuyo_${prefix}_joint" type="revolute">
+	<!-- joint for laser platform  -->
+	<joint name="laser_tilt_mount_joint" type="fixed">
 	     <axis xyz="0 1 0" />
 	     <origin xyz="${origin_x} 0 ${origin_z}" rpy="0 0 ${origin_yaw}" />
 	     <parent link="${parent}"/>
+	     <child link="laser_tilt_mount_link"/>
+	     <limit effort="30" lower="-2.6" upper="2.6" velocity="2.0"/>
+		 <dynamics damping="100"/>
+	</joint>
+	<link name="laser_tilt_mount_link">
+	     <inertial>
+	  		<origin xyz="0 0 0" rpy="0 0 0"/>
+	  		<mass value="1"/>
+		 <inertia ixx="1.0" ixy="0.0" ixz="0.0" iyy="1.0" iyz="0.0" izz="1.0"/></inertial>
+	</link>
+	<!-- joint for laser platform rotation -->
+	<joint name="hokuyo_${prefix}_joint" type="revolute">
+	    <axis xyz="0 1 0" />
+	    <origin xyz="0 0 0" rpy="0 0 0" />
+	    <parent link="laser_tilt_mount_link"/>
+	    <child link="laser_tilt_link"/> <!-- hokuyo_${prefix}_link -->
+	    <limit effort="${ptz_joint_effort_limit}" velocity="${ptz_joint_velocity_limit}" lower="-1.5708" upper="1.5708"/>
+	    <joint_properties damping="${ptz_joint_damping}" friction="{ptz_joint_friction}"/>
+	</joint>
+	<!-- transmission -->
+	<transmission name="joint_${prefix}_trans">
+	  <type>transmission_interface/SimpleTransmission</type>
+	    <joint name="hokuyo_${prefix}_joint" />
+	    <actuator name="${prefix}_motor">
+	       <hardwareInterface>EffortJointInterface</hardwareInterface>
+	       <mechanicalReduction>${ptz_mechanical_reduction}</mechanicalReduction>
+	    </actuator>
+	</transmission>
+	<link name="laser_tilt_link">
+	   <inertial>
+	     <mass value="0.1" />
+	     <origin xyz="0 0 0" rpy="0 0 0" />
+	     <inertia ixx="0.1" ixy="0" ixz="0" iyy="0.1" iyz="0" izz="0.1" />
+	     <!-- <inertia ixx="1e-6" ixy="0" ixz="0" iyy="1e-6" iyz="0" izz="1e-6" /> -->
+	  </inertial>
+	</link>
+	<!--  HOKUYO FRONTAL SENSOR joint -->
+	<joint name="hokuyo_frontal_laser_joint" type="fixed">
+	     <axis xyz="0 1 0" />
+	     <origin xyz="0.021 0 ${laser_offset_z}"/>
+	     <parent link="laser_tilt_link"/>
 	     <child link="hokuyo_${prefix}_link"/>
-	     <limit effort="${ptz_joint_effort_limit}" velocity="${ptz_joint_velocity_limit}" lower="-1.5708" upper="1.5708"/>
-	     <joint_properties damping="${ptz_joint_damping}" friction="{ptz_joint_friction}"/>
-	  </joint>
- 	<!-- link -->
-	  <link name="hokuyo_${prefix}_link">
-	     <inertial>
-	       <mass value="0.1" />
-	       <origin xyz="0 0 0" rpy="0 0 0" />
-	       <inertia ixx="0.1" ixy="0" ixz="0" iyy="0.1" iyz="0" izz="0.1" />
-	       <!-- <inertia ixx="1e-6" ixy="0" ixz="0" iyy="1e-6" iyz="0" izz="1e-6" /> -->
-	    </inertial>
-	  </link>
- 	<!-- transmission -->
-	 <transmission name="joint_${prefix}_trans">
-	   <type>transmission_interface/SimpleTransmission</type>
-	     <joint name="hokuyo_${prefix}_joint" />
-	     <actuator name="${prefix}_motor">
-	     <hardwareInterface>EffortJointInterface</hardwareInterface>
-	       <mechanicalReduction>${ptz_mechanical_reduction}</mechanicalReduction>
-	     </actuator>
-	 </transmission>
-	<!-- gazebo -->
-	 <gazebo reference="hokuyo_${prefix}_link">
+	</joint>
+	<!-- HOKUYO FRONTAL SENSOR link -->
+	<link name="hokuyo_${prefix}_link">
+	   <inertial>
+	     <mass value="0.1" />
+	     <origin xyz="0 0 0" rpy="0 0 0" />
+	     <inertia ixx="0.1" ixy="0" ixz="0" iyy="0.1" iyz="0" izz="0.1" />
+	<!--      <inertia ixx="1e-6" ixy="0" ixz="0" iyy="1e-6" iyz="0" izz="1e-6" /> -->
+	  </inertial>
+	</link>
+	<!-- GAZEBO properties and plugins -->
+	<gazebo reference="hokuyo_${prefix}_link">
 	    <material>Gazebo/Grey</material>
 	    <sensor type="ray" name="${prefix}_sensor">
@@ -70,5 +101,5 @@
 	      </plugin>
 	    </sensor>
-	 </gazebo>
+	</gazebo>
   </xacro:macro>
 </robot>
