Commit message: Uniformization of tf names

File: guardian_sim/guardian_description/urdf/guardian_base.urdf.xacro (robot description, xacro)
@@ -53,5 +53,5 @@
 		<sensor_imu parent="base_link" /> <!-- guardian_robot_control uses imu to update odometry -->
 		<sensor_hokuyo_front parent="base_link" prefix="tilt_laser" visualize="true" origin_x="0.46781" origin_z="0.24299" origin_yaw="0" />
-		<sensor_hokuyo_back parent="base_link" prefix="base_laser" visualize="true" origin_x="-0.4323" origin_z="0.3" origin_yaw="${PI}" />
+		<sensor_hokuyo_back parent="base_link" prefix="back_laser" visualize="true" origin_x="-0.4323" origin_z="0.3" origin_yaw="${PI}" />
 	</xacro:macro>
 </robot>

File: guardian_sim/guardian_description/urdf/sensors/hokuyo_front.urdf.xacro (robot description, xacro)
@@ -56,8 +56,8 @@
 	     <origin xyz="0.021 0 ${laser_offset_z}"/>
 	     <parent link="laser_tilt_link"/>
-	     <child link="hokuyo_${prefix}_link"/>
+	     <child link="hokuyo_frontal_laser_link"/>
 	</joint>
 	<!-- HOKUYO FRONTAL SENSOR link -->
-	<link name="hokuyo_${prefix}_link">
+	<link name="hokuyo_frontal_laser_link">
 	   <inertial>
 	     <mass value="0.1" />
@@ -68,5 +68,5 @@
 	</link>
 	<!-- GAZEBO properties and plugins -->
-	<gazebo reference="hokuyo_${prefix}_link">
+	<gazebo reference="hokuyo_frontal_laser_link">
 	    <material>Gazebo/Grey</material>
 	    <sensor type="ray" name="${prefix}_sensor">
@@ -96,5 +96,5 @@
 	      <plugin name="${prefix}_plugin" filename="libgazebo_ros_laser_2D.so">
 	        <topicName>/guardian/laser_tilt_front</topicName>
-	        <frameName>hokuyo_${prefix}_link</frameName>
+	        <frameName>hokuyo_frontal_laser_link</frameName>
 	        <time_increment>0.00009765739</time_increment> <!-- time between measurements --> <!-- 0.0667 sec /683 steps -->
 	        <intensities>0</intensities> <!-- Whether or not the hokuyo laser returns intensity values. 0 means no intensities[] -->

Commit message: Changed tilt laser and kinect orientation to look at the ceiling of the ship_interior.

File: guardian_sim/guardian_description/urdf/guardian_base.urdf.xacro (robot description, xacro)
@@ -52,6 +52,6 @@
 		<sensor_kinect parent="base_link"/>
 		<sensor_imu parent="base_link" /> <!-- guardian_robot_control uses imu to update odometry -->
-		<sensor_hokuyo_front parent="base_link" prefix="tilt_laser" visualize="true" origin_x="0.46781" origin_z="0.24299" origin_yaw="0" />
-		<sensor_hokuyo_back parent="base_link" prefix="back_laser" visualize="true" origin_x="-0.4323" origin_z="0.3" origin_yaw="${PI}" />
+		<sensor_hokuyo_front parent="base_link" prefix="tilt_laser" visualize="true" origin_x="0.46781" origin_y="0.0" origin_z="0.24299" origin_roll="0.0" origin_pitch="0.0" origin_yaw="0" />
+		<sensor_hokuyo_back parent="base_link" prefix="back_laser" visualize="true" origin_x="-0.4323" origin_y="0.0" origin_z="0.3" origin_roll="0.0" origin_pitch="0.0" origin_yaw="${PI}" />
 	</xacro:macro>
 </robot>

File: guardian_sim/guardian_description/urdf/sensors/hokuyo_back.urdf.xacro (robot description, xacro)
@@ -8,9 +8,9 @@
 	<xacro:property name="ptz_joint_damping" value="0.1" />
 	<xacro:property name="ptz_mechanical_reduction" value="1.0" />
-	<xacro:macro name="sensor_hokuyo_back" params="parent prefix visualize origin_x origin_z origin_yaw">
+	<xacro:macro name="sensor_hokuyo_back" params="parent prefix visualize origin_x origin_y origin_z origin_roll origin_pitch origin_yaw">
 		<!-- joint -->
 		<joint name="hokuyo_${prefix}_joint" type="fixed">
 			<axis xyz="0 1 0" />
-			<origin xyz="${origin_x} 0 ${origin_z}" rpy="0 0 ${origin_yaw}" />
+			<origin xyz="${origin_x} ${origin_y} ${origin_z}" rpy="${origin_roll} ${origin_pitch} ${origin_yaw}" />
 			<parent link="${parent}" />
 			<child link="hokuyo_${prefix}_link" />

File: guardian_sim/guardian_description/urdf/sensors/hokuyo_front.urdf.xacro (robot description, xacro)
@@ -9,9 +9,9 @@
   <xacro:property name="ptz_mechanical_reduction" value="1.0" />
   <xacro:property name="laser_offset_z" value="0.06" />
-  <xacro:macro name="sensor_hokuyo_front" params="parent prefix visualize origin_x origin_z origin_yaw">
+  <xacro:macro name="sensor_hokuyo_front" params="parent prefix visualize origin_x origin_y origin_z origin_roll origin_pitch origin_yaw">
 	<!-- joint for laser platform  -->
 	<joint name="laser_tilt_mount_joint" type="fixed">
 	     <axis xyz="0 1 0" />
-	     <origin xyz="${origin_x} 0 ${origin_z}" rpy="0 0 ${origin_yaw}" />
+	     <origin xyz="${origin_x} ${origin_y} ${origin_z}" rpy="${origin_roll} ${origin_pitch} ${origin_yaw}" />
 	     <parent link="${parent}"/>
 	     <child link="laser_tilt_mount_link"/>

File: guardian_sim/guardian_description/urdf/sensors/kinect_properties.urdf.xacro (robot description, xacro)
@@ -6,5 +6,5 @@
 	<property name="cam_pz" value="0.423" />
 	<property name="cam_or" value="0" />
-	<property name="cam_op" value="0" />
+	<property name="cam_op" value="-0.78539816339" />
 	<property name="cam_oy" value="0" />
 </robot>

File: guardian_sim/guardian_description/urdf/wheel.urdf.xacro (robot description, xacro)
@@ -27,4 +27,7 @@
 					<mesh filename="package://guardian_description/meshes/wheel.stl" />
 				</geometry>
+				<material name="grey">
+					<color rgba="0.2 0.2 0.2 1.0" />
+				</material>
 			</visual>
 			<collision>

Commit message: Revision and correction of all robots TFs. Added TFs for Structure IO 3D sensor and projetor.

File: guardian_sim/guardian_description/urdf/guardian_base.urdf.xacro (robot description, xacro)
@@ -6,5 +6,5 @@
 	<xacro:include filename="$(find guardian_description)/urdf/sensors/hokuyo_front.urdf.xacro" />
 	<xacro:include filename="$(find guardian_description)/urdf/sensors/hokuyo_back.urdf.xacro" />
-	<xacro:macro name="guardian_base" params="base_footprint_z">
+	<xacro:macro name="guardian_base" params="base_footprint_z use_simulated_kinect">
 		<!-- BASE FOOTPRINT -->
 		<!-- base_footprint is a fictitious link(frame) that is on the ground right below base_link origin, navigation stack depends on this frame -->
@@ -25,6 +25,25 @@
 			<child link="base_link" />
 		</joint>
+		<!-- kinect and projector metal support -->
+		<link name="support_bottom_link" />
+		<joint name="support_bottom_joint" type="fixed">
+			<origin xyz="0.185 0 0.2305" rpy="0 0 0" />
+			<parent link="base_link" />
+			<child link="support_bottom_link" />
+		</joint>
+		<link name="support_top_link" />
+		<joint name="support_top_joint" type="fixed">
+			<origin xyz="0.184 0 0.267" rpy="0 0 0" />
+			<parent link="support_bottom_link" />
+			<child link="support_top_link" />
+		</joint>
+		<link name="projector_link" />
+		<joint name="projector_joint" type="fixed">
+			<origin xyz="-0.06 -0.031 -0.041" rpy="0 0 0" />
+			<parent link="support_top_link" />
+			<child link="projector_link" />
+		</joint>
 		<!-- BASE_LINK (Grey) -->
-		<link name="base_link">
+		<link name="base_link"> <!-- center of wheels -> rotation axis -->
 			<inertial>
 				<mass value="95.0" /> <!-- 95.0 -->
@@ -50,8 +69,24 @@
 		</link>
 		<!-- ################# SENSORS ################# -->
-		<sensor_kinect parent="base_link"/>
+		<xacro:if value="${use_simulated_kinect}">
+ 			<sensor_kinect parent="base_link"/>
+		</xacro:if>
+		<xacro:unless value="${use_simulated_kinect}">
+			<link name="camera_link_support_axis" />
+			<joint name="camera_link_support_axis_joint" type="fixed">
+				<origin xyz="-0.015 0.015 0.0" rpy="1.565 0.4025 0.02" />
+				<parent link="support_top_link" />
+				<child link="camera_link_support_axis" />
+			</joint>
+			<link name="camera_link" />
+			<joint name="camera_link_joint" type="fixed">
+				<origin xyz="0.05 0.057 -0.016" rpy="0 0 0" />
+				<parent link="camera_link_support_axis" />
+				<child link="camera_link" />
+			</joint>
+		</xacro:unless>
 		<sensor_imu parent="base_link" /> <!-- guardian_robot_control uses imu to update odometry -->
-		<sensor_hokuyo_front parent="base_link" prefix="tilt_laser" visualize="true" origin_x="0.45" origin_y="0.025" origin_z="0.24299" origin_roll="-0.01" origin_pitch="0.03" origin_yaw="-0.02" />
-		<sensor_hokuyo_back parent="base_link" prefix="back_laser" visualize="true" origin_x="-0.43" origin_y="-0.015" origin_z="0.3" origin_roll="0.03" origin_pitch="-0.015" origin_yaw="${PI}" />
+		<sensor_hokuyo_front parent="base_link" prefix="front_laser" visualize="true" origin_x="0.46" origin_y="-0.0025" origin_z="0.2595" origin_roll="0.0" origin_pitch="0.0" origin_yaw="-0.026" />
+		<sensor_hokuyo_back parent="base_link" prefix="back_laser" visualize="true" origin_x="-0.433" origin_y="-0.0085" origin_z="0.3065" origin_roll="0.0" origin_pitch="0.0" origin_yaw="${PI}" />
 	</xacro:macro>
 </robot>

File: guardian_sim/guardian_description/urdf/guardian_tracks.urdf.xacro (robot description, xacro)
@@ -5,5 +5,5 @@
 	<xacro:include filename="$(find guardian_description)/urdf/track_wheel.urdf.xacro" />
 	<!-- ###### BASE ###### -->
-	<guardian_base base_footprint_z="0.069" />
+	<guardian_base base_footprint_z="0.0635" use_simulated_kinect="false" />
 	<!-- ###### TRACKS ###### -->
 	<!-- visual -->

File: guardian_sim/guardian_description/urdf/guardian_wheels.urdf.xacro (robot description, xacro)
@@ -2,10 +2,10 @@
 <robot name="guardian" xmlns:xacro="http://www.ros.org/wiki/xacro">
 	<xacro:property name="wheelSeparation" value="0.612" />
-	<xacro:property name="wheelDiameter" value="0.37" />
+	<xacro:property name="wheelDiameter" value="0.35" />
 	<xacro:include filename="$(find guardian_description)/urdf/guardian_base.urdf.xacro" />
 	<xacro:include filename="$(find guardian_description)/urdf/track.urdf.xacro" />
 	<xacro:include filename="$(find guardian_description)/urdf/wheel.urdf.xacro" />
 	<!-- ###### BASE ###### -->
-	<guardian_base base_footprint_z="0.165" />
+	<guardian_base base_footprint_z="0.175" use_simulated_kinect="false" /> <!-- wheels radius -->
 	<!-- ###### TRACKS ###### -->
 	<track parent="base_link" prefix="left_track" joint_yaw="${PI}" />

File: guardian_sim/guardian_description/urdf/old_files/guardian_wheels_laser_up.urdf.xacro (robot description, xacro)
@@ -390,8 +390,8 @@
      <origin xyz="${laser_offset_x+0.066} 0 ${laser_offset_z}"/>
      <parent link="laser_tilt_link"/>
-     <child link="hokuyo_frontal_laser_link"/>
+     <child link="hokuyo_front_laser_link"/>
   </joint>
   <!-- Hokuyo Laser -->
-  <link name="hokuyo_frontal_laser_link">
+  <link name="hokuyo_front_laser_link">
     <collision>
       <origin xyz="0 0 0" rpy="0 0 0"/>

File: guardian_sim/guardian_description/urdf/sensors/hokuyo_front.urdf.xacro (robot description, xacro)
@@ -1,105 +1,101 @@
 <?xml version="1.0"?>
 <robot xmlns:xacro="http://www.ros.org/wiki/xacro">
-  <!-- Robot parameters -->
-  <xacro:property name="PI" value="3.1415926535897931"/>
-  <xacro:property name="ptz_joint_effort_limit" value="100.0" />
-  <xacro:property name="ptz_joint_velocity_limit" value="100.0"/>
-  <xacro:property name="ptz_joint_friction" value="0.1" />
-  <xacro:property name="ptz_joint_damping" value="0.1" />
-  <xacro:property name="ptz_mechanical_reduction" value="1.0" />
-  <xacro:property name="laser_offset_z" value="0.06" />
-  <xacro:macro name="sensor_hokuyo_front" params="parent prefix visualize origin_x origin_y origin_z origin_roll origin_pitch origin_yaw">
-	<!-- joint for laser platform  -->
-	<joint name="laser_tilt_mount_joint" type="fixed">
-	     <axis xyz="0 1 0" />
-	     <origin xyz="${origin_x} ${origin_y} ${origin_z}" rpy="${origin_roll} ${origin_pitch} ${origin_yaw}" />
-	     <parent link="${parent}"/>
-	     <child link="laser_tilt_mount_link"/>
-	     <limit effort="30" lower="-2.6" upper="2.6" velocity="2.0"/>
-		 <dynamics damping="100"/>
-	</joint>
-	<link name="laser_tilt_mount_link">
-	     <inertial>
-	  		<origin xyz="0 0 0" rpy="0 0 0"/>
-	  		<mass value="1"/>
-		 <inertia ixx="1.0" ixy="0.0" ixz="0.0" iyy="1.0" iyz="0.0" izz="1.0"/></inertial>
-	</link>
-	<!-- joint for laser platform rotation -->
-	<joint name="hokuyo_${prefix}_joint" type="revolute">
-	    <axis xyz="0 1 0" />
-	    <origin xyz="0 0 0" rpy="0 0 0" />
-	    <parent link="laser_tilt_mount_link"/>
-	    <child link="laser_tilt_link"/> <!-- hokuyo_${prefix}_link -->
-	    <limit effort="${ptz_joint_effort_limit}" velocity="${ptz_joint_velocity_limit}" lower="-1.5708" upper="1.5708"/>
-	    <joint_properties damping="${ptz_joint_damping}" friction="{ptz_joint_friction}"/>
-	</joint>
-	<!-- transmission -->
-	<transmission name="joint_${prefix}_trans">
-	  <type>transmission_interface/SimpleTransmission</type>
-	    <joint name="hokuyo_${prefix}_joint" />
-	    <actuator name="${prefix}_motor">
-	       <hardwareInterface>EffortJointInterface</hardwareInterface>
-	       <mechanicalReduction>${ptz_mechanical_reduction}</mechanicalReduction>
-	    </actuator>
-	</transmission>
-	<link name="laser_tilt_link">
-	   <inertial>
-	     <mass value="0.1" />
-	     <origin xyz="0 0 0" rpy="0 0 0" />
-	     <inertia ixx="0.1" ixy="0" ixz="0" iyy="0.1" iyz="0" izz="0.1" />
-	     <!-- <inertia ixx="1e-6" ixy="0" ixz="0" iyy="1e-6" iyz="0" izz="1e-6" /> -->
-	  </inertial>
-	</link>
-	<!--  HOKUYO FRONTAL SENSOR joint -->
-	<joint name="hokuyo_frontal_laser_joint" type="fixed">
-	     <axis xyz="0 1 0" />
-	     <origin xyz="0.021 0 ${laser_offset_z}"/>
-	     <parent link="laser_tilt_link"/>
-	     <child link="hokuyo_frontal_laser_link"/>
-	</joint>
-	<!-- HOKUYO FRONTAL SENSOR link -->
-	<link name="hokuyo_frontal_laser_link">
-	   <inertial>
-	     <mass value="0.1" />
-	     <origin xyz="0 0 0" rpy="0 0 0" />
-	     <inertia ixx="0.1" ixy="0" ixz="0" iyy="0.1" iyz="0" izz="0.1" />
-	<!--      <inertia ixx="1e-6" ixy="0" ixz="0" iyy="1e-6" iyz="0" izz="1e-6" /> -->
-	  </inertial>
-	</link>
-	<!-- GAZEBO properties and plugins -->
-	<gazebo reference="hokuyo_frontal_laser_link">
-	    <material>Gazebo/Grey</material>
-	    <sensor type="ray" name="${prefix}_sensor">
-	      <pose>0 0 0 0 0 0</pose>
-	      <visualize>${visualize}</visualize>
-	      <update_rate>10</update_rate> <!-- rate of 10 for scan time ~ 100 ms  -->
-	      <ray>
-	        <scan>
-	          <horizontal>
-	           <samples>684</samples> <!-- 683 steps + 1 -->
-	           <resolution>1</resolution>
-	           <min_angle>-2.0943951</min_angle>   <!-- 240 deg (total) in the front -->
-	           <max_angle>2.0943951</max_angle>
-	          </horizontal>
-	        </scan>
-	        <range>
-	          <min>0.10</min>
-	          <max>5.0</max> <!-- 5.0 -->
-	          <resolution>0.001</resolution> <!-- 0.001 -->
-	        </range>
-	        <noise>
-	          <type>gaussian</type>
-	          <mean>0.0</mean>
-	          <stddev>0.0033</stddev> <!-- 0.0033 -->
-	        </noise>
-	      </ray>
-	      <plugin name="${prefix}_plugin" filename="libgazebo_ros_laser_2D.so">
-	        <topicName>/guardian/laser_tilt_front</topicName>
-	        <frameName>hokuyo_frontal_laser_link</frameName>
-	        <time_increment>0.00009765739</time_increment> <!-- time between measurements --> <!-- 0.0667 sec /683 steps -->
-	        <intensities>0</intensities> <!-- Whether or not the hokuyo laser returns intensity values. 0 means no intensities[] -->
-	      </plugin>
-	    </sensor>
-	</gazebo>
-  </xacro:macro>
+	<!-- Robot parameters -->
+	<xacro:property name="PI" value="3.1415926535897931" />
+	<xacro:property name="ptz_joint_effort_limit" value="30.0" />
+	<xacro:property name="ptz_joint_velocity_limit" value="2.0" />
+	<xacro:property name="ptz_joint_friction" value="0.1" />
+	<xacro:property name="ptz_joint_damping" value="0.1" />
+	<xacro:property name="ptz_mechanical_reduction" value="1.0" />
+	<xacro:macro name="sensor_hokuyo_front" params="parent prefix visualize origin_x origin_y origin_z origin_roll origin_pitch origin_yaw"> <!-- origin -> laser rotation axis center -->
+		<!-- front laser tilting platform -->
+		<link name="hokuyo_${prefix}_tilt_support_link" >
+			<inertial>
+				<origin xyz="0 0 0" rpy="0 0 0" />
+				<mass value="0.3" />
+				<inertia ixx="1.0" ixy="0.0" ixz="0.0" iyy="1.0" iyz="0.0" izz="1.0" />
+			</inertial>
+		</link>
+		<joint name="hokuyo_${prefix}_tilt_support_joint" type="fixed">
+			<axis xyz="0 1 0" />
+			<origin xyz="${origin_x} ${origin_y} ${origin_z}" rpy="${origin_roll} ${origin_pitch} ${origin_yaw}" />
+			<parent link="${parent}" />
+			<child link="hokuyo_${prefix}_tilt_support_link" />
+			<limit effort="30" lower="-2.6" upper="2.6" velocity="2.0"/>
+		 	<dynamics damping="100"/>
+		</joint>
+		<!-- front laser tilting platform motor -->
+		<link name="hokuyo_${prefix}_tilt_axis_link" >
+			<inertial>
+				<origin xyz="0 0 0" rpy="0 0 0" />
+				<mass value="1" />
+				<inertia ixx="0.1" ixy="0" ixz="0" iyy="0.1" iyz="0" izz="0.1" />
+			</inertial>
+		</link>
+		<joint name="hokuyo_${prefix}_tilt_joint" type="revolute">
+			<axis xyz="0 1 0" />
+			<origin xyz="0 0 0" rpy="0 0 0" />
+			<parent link="hokuyo_${prefix}_tilt_support_link" />
+			<child link="hokuyo_${prefix}_tilt_axis_link" />
+			<limit effort="${ptz_joint_effort_limit}" velocity="${ptz_joint_velocity_limit}" lower="-1.5708" upper="1.5708" />
+			<joint_properties damping="${ptz_joint_damping}" friction="{ptz_joint_friction}" />
+		</joint>
+		<transmission name="joint_${prefix}_trans">
+			<type>transmission_interface/SimpleTransmission</type>
+			<joint name="hokuyo_${prefix}_joint" />
+			<actuator name="${prefix}_motor">
+				<hardwareInterface>EffortJointInterface</hardwareInterface>
+				<mechanicalReduction>${ptz_mechanical_reduction}</mechanicalReduction>
+			</actuator>
+		</transmission>
+		<!-- front laser -->
+		<joint name="hokuyo_${prefix}_joint" type="fixed">
+			<axis xyz="0 1 0" />
+			<origin xyz="0.026 -0.0015 0.0565" />
+			<parent link="hokuyo_${prefix}_tilt_axis_link" />
+			<child link="hokuyo_${prefix}_link" />
+		</joint>
+		<link name="hokuyo_${prefix}_link">
+			<inertial>
+				<mass value="0.1" />
+				<origin xyz="0 0 0" rpy="0 0 0" />
+				<inertia ixx="0.1" ixy="0" ixz="0" iyy="0.1" iyz="0" izz="0.1" />
+			</inertial>
+		</link>
+		<!-- GAZEBO properties and plugins -->
+		<gazebo reference="hokuyo_${prefix}_link">
+			<material>Gazebo/Grey</material>
+			<sensor type="ray" name="${prefix}_sensor">
+				<pose>0 0 0 0 0 0</pose>
+				<visualize>${visualize}</visualize>
+				<update_rate>10</update_rate> <!-- rate of 10 for scan time ~ 100 ms -->
+				<ray>
+					<scan>
+						<horizontal>
+							<samples>684</samples> <!-- 683 steps + 1 -->
+							<resolution>1</resolution>
+							<min_angle>-2.0943951</min_angle>   <!-- 240 deg (total) in the front -->
+							<max_angle>2.0943951</max_angle>
+						</horizontal>
+					</scan>
+					<range>
+						<min>0.10</min>
+						<max>5.0</max> <!-- 5.0 -->
+						<resolution>0.001</resolution> <!-- 0.001 -->
+					</range>
+					<noise>
+						<type>gaussian</type>
+						<mean>0.0</mean>
+						<stddev>0.0033</stddev> <!-- 0.0033 -->
+					</noise>
+				</ray>
+				<plugin name="${prefix}_plugin" filename="libgazebo_ros_laser_2D.so">
+					<topicName>/guardian/laser_tilt_front</topicName>
+					<frameName>hokuyo_${prefix}_link</frameName>
+					<time_increment>0.00009765739</time_increment> <!-- time between measurements --> <!-- 0.0667 sec /683 steps -->
+					<intensities>0</intensities> <!-- Whether or not the hokuyo laser returns intensity values. 0 means no intensities[] -->
+				</plugin>
+			</sensor>
+		</gazebo>
+	</xacro:macro>
 </robot>

File: guardian_sim/guardian_description/urdf/wheel.urdf.xacro (robot description, xacro)
@@ -4,5 +4,5 @@
 	<xacro:property name="mass" value="4.3" />
 	<xacro:property name="simple_wheel_length" value="0.1143" />
-	<xacro:property name="simple_wheel_radius" value="0.1850" />
+	<xacro:property name="simple_wheel_radius" value="0.175" />
 	<xacro:property name="wheel_origin_y" value="0.03" />
 	<xacro:property name="wheel_offset_x" value="0.300" />

Commit message: Updated kinect tf to new position on robot metal support.

File: guardian_sim/guardian_description/urdf/guardian_base.urdf.xacro (robot description, xacro)
@@ -34,14 +34,14 @@
 		<link name="support_top_link" />
 		<joint name="support_top_joint" type="fixed">
-			<origin xyz="0.184 0 0.267" rpy="0 0 0" />
+			<origin xyz="0.31 0 0.265" rpy="0 0 0" />
 			<parent link="support_bottom_link" />
 			<child link="support_top_link" />
 		</joint>
-		<link name="projector_link" />
+		<!-- <link name="projector_link" />
 		<joint name="projector_joint" type="fixed">
-			<origin xyz="-0.06 -0.031 -0.041" rpy="0 0 0" />
+			<origin xyz="-0.07 0.031 -0.041" rpy="1.5707 0 0" />
 			<parent link="support_top_link" />
 			<child link="projector_link" />
-		</joint>
+		</joint> -->
 		<!-- BASE_LINK (Grey) -->
 		<link name="base_link"> <!-- center of wheels -> rotation axis -->
@@ -75,5 +75,5 @@
 			<link name="camera_link_support_axis" />
 			<joint name="camera_link_support_axis_joint" type="fixed">
-				<origin xyz="-0.015 0.015 0.0" rpy="1.565 0.4025 0.02" />
+				<origin xyz="-0.027 -0.015 0.0" rpy="1.565 0.5675 0.02" />
 				<parent link="support_top_link" />
 				<child link="camera_link_support_axis" />
@@ -81,5 +81,5 @@
 			<link name="camera_link" />
 			<joint name="camera_link_joint" type="fixed">
-				<origin xyz="0.05 0.057 -0.016" rpy="0 0 0" />
+				<origin xyz="0.06 0.057 0.016" rpy="0 0 0" />
 				<parent link="camera_link_support_axis" />
 				<child link="camera_link" />

Commit message: Updated robot TFs.

File: guardian_sim/guardian_description/urdf/guardian_base.urdf.xacro (robot description, xacro)
@@ -28,5 +28,5 @@
 		<link name="support_bottom_link" />
 		<joint name="support_bottom_joint" type="fixed">
-			<origin xyz="0.185 0 0.2305" rpy="0 0 0" />
+			<origin xyz="0.185 0 0.2425" rpy="0 0 0" />
 			<parent link="base_link" />
 			<child link="support_bottom_link" />
@@ -34,5 +34,5 @@
 		<link name="support_top_link" />
 		<joint name="support_top_joint" type="fixed">
-			<origin xyz="0.31 0 0.265" rpy="0 0 0" />
+			<origin xyz="0.314 0.0 0.256" rpy="0 0 0" />
 			<parent link="support_bottom_link" />
 			<child link="support_top_link" />
@@ -75,5 +75,5 @@
 			<link name="camera_link_support_axis" />
 			<joint name="camera_link_support_axis_joint" type="fixed">
-				<origin xyz="-0.027 -0.015 0.0" rpy="1.565 0.5675 0.02" />
+				<origin xyz="0.0 -0.015 0.0" rpy="1.565 0.60 0.05" />
 				<parent link="support_top_link" />
 				<child link="camera_link_support_axis" />
@@ -81,5 +81,5 @@
 			<link name="camera_link" />
 			<joint name="camera_link_joint" type="fixed">
-				<origin xyz="0.06 0.057 0.016" rpy="0 0 0" />
+				<origin xyz="0.045 0.065 0.0155" rpy="0 0 0" />
 				<parent link="camera_link_support_axis" />
 				<child link="camera_link" />
