Commit message: Added IMUs (MPU-9150 and UM7) frames to guardian xacro.

File: guardian_sim/guardian_description/urdf/guardian_base.urdf.xacro (robot description, xacro)
@@ -34,5 +34,5 @@
 		<link name="support_top_link" />
 		<joint name="support_top_joint" type="fixed">
-			<origin xyz="0.314 0.0 0.256" rpy="0 0 0" />
+			<origin xyz="0.29 0.0 0.26" rpy="0.0 0 -0.05" />
 			<parent link="support_bottom_link" />
 			<child link="support_top_link" />
@@ -75,5 +75,5 @@
 			<link name="camera_link_support_axis" />
 			<joint name="camera_link_support_axis_joint" type="fixed">
-				<origin xyz="0.0 -0.015 0.0" rpy="1.565 0.60 0.05" />
+				<origin xyz="0.0 -0.015 0.0" rpy="1.565 0.619 0.05" />
 				<parent link="support_top_link" />
 				<child link="camera_link_support_axis" />

File: guardian_sim/guardian_description/urdf/sensors/imu.urdf.xacro (robot description, xacro)
@@ -1,43 +1,49 @@
 <?xml version="1.0"?>
 <robot xmlns:xacro="http://www.ros.org/wiki/xacro">
-  <xacro:property name="PI" value="3.1415926535897931"/>
-  <xacro:macro name="sensor_imu" params="parent">
-	<!-- joint -->
-	  <joint name="imu_joint" type="fixed">
-	      <axis xyz="1 0 0"/> <!-- 0 1 0 -->
-	      <origin xyz="0 0 0.2825"/>
-	      <parent link="${parent}"/>
-	      <child link="imu_link"/>
-	  </joint>
- 	<!-- link -->
-	  <link name="imu_link">
-	      <inertial>
-	        <mass value="0.001"/>
-	        <origin rpy="0 0 0" xyz="0 0 0"/>
-	        <inertia ixx="0.0001" ixy="0" ixz="0" iyy="0.000001" iyz="0" izz="0.0001"/>
-	      </inertial>
-	      <visual>
-	        <origin rpy="0 0 0" xyz="0 0 0"/>
-	        <geometry>
-	          <box size="0.001 0.001 0.001"/>
-	        </geometry>
-	      </visual>
-	      <collision>
-	        <origin rpy="0 0 0" xyz="0 0 0"/>
-	        <geometry>
-	          <box size=".001 .001 .001"/>
-	        </geometry>
-	      </collision>
-	  </link>
- 	<!-- plugin -->
-	  <gazebo>
-	    <plugin name="ros_imu" filename="libgazebo_ros_imu.so">
-	       <robotNamespace>/guardian</robotNamespace>
-	       <topicName>imu_data</topicName>
-			<bodyName>imu_link </bodyName>
-			<serviceName>/imu_service</serviceName>
-	        <gaussianNoise>0.005</gaussianNoise>
-	    </plugin>
-	  </gazebo>
-  </xacro:macro>
+	<xacro:property name="PI" value="3.1415926535897931" />
+	<xacro:macro name="sensor_imu" params="parent">
+		<!-- joint -->
+		<joint name="imu_mpu_9150_joint" type="fixed">
+			<axis xyz="1 0 0" /> <!-- 0 1 0 -->
+			<origin xyz="0.0775 0.0 0.1555" rpy="0 0 0 " />
+			<parent link="${parent}" />
+			<child link="imu_mpu_9150_link" />
+		</joint>
+		<!-- link -->
+		<link name="imu_mpu_9150_link">
+			<inertial>
+				<mass value="0.001" />
+				<origin rpy="0 0 0" xyz="0 0 0" />
+				<inertia ixx="0.0001" ixy="0" ixz="0" iyy="0.000001" iyz="0" izz="0.0001" />
+			</inertial>
+			<visual>
+				<origin rpy="0 0 0" xyz="0 0 0" />
+				<geometry>
+					<box size="0.001 0.001 0.001" />
+				</geometry>
+			</visual>
+			<collision>
+				<origin rpy="0 0 0" xyz="0 0 0" />
+				<geometry>
+					<box size=".001 .001 .001" />
+				</geometry>
+			</collision>
+		</link>
+		<!-- plugin -->
+		<gazebo>
+			<plugin name="ros_imu" filename="libgazebo_ros_imu.so">
+				<robotNamespace>/guardian</robotNamespace>
+				<topicName>imu_data</topicName>
+				<bodyName>imu_link </bodyName>
+				<serviceName>/imu_service</serviceName>
+				<gaussianNoise>0.005</gaussianNoise>
+			</plugin>
+		</gazebo>
+		<link name="imu_um7_link" />
+		<joint name="imu_um7_joint" type="fixed">
+			<origin xyz="0.056 0.0 0.1355" rpy="0 0 0 " />
+			<parent link="${parent}" />
+			<child link="imu_um7_link" />
+		</joint>
+	</xacro:macro>
 </robot>

Commit message: Updated TFs for struture io.

File: guardian_sim/guardian_description/urdf/guardian_base.urdf.xacro (robot description, xacro)
@@ -34,5 +34,5 @@
 		<link name="support_top_link" />
 		<joint name="support_top_joint" type="fixed">
-			<origin xyz="0.29 0.0 0.26" rpy="0.0 0 -0.05" />
+			<origin xyz="0.314 0.0 0.256" rpy="0.0 0 0.0" />
 			<parent link="support_bottom_link" />
 			<child link="support_top_link" />
@@ -75,5 +75,5 @@
 			<link name="camera_link_support_axis" />
 			<joint name="camera_link_support_axis_joint" type="fixed">
-				<origin xyz="0.0 -0.015 0.0" rpy="1.565 0.619 0.05" />
+				<origin xyz="-0.02 -0.015 0.0" rpy="1.5708 0.619 0.0" />
 				<parent link="support_top_link" />
 				<child link="camera_link_support_axis" />
@@ -81,5 +81,5 @@
 			<link name="camera_link" />
 			<joint name="camera_link_joint" type="fixed">
-				<origin xyz="0.045 0.065 0.0155" rpy="0 0 0" />
+				<origin xyz="0.045 0.06 0.017" rpy="0 0 0" />
 				<parent link="camera_link_support_axis" />
 				<child link="camera_link" />

Commit message: Updated TFs for kinect and front laser.

File: guardian_sim/guardian_description/urdf/guardian_base.urdf.xacro (robot description, xacro)
@@ -75,5 +75,5 @@
 			<link name="camera_link_support_axis" />
 			<joint name="camera_link_support_axis_joint" type="fixed">
-				<origin xyz="-0.02 -0.015 0.0" rpy="1.5708 0.619 0.0" />
+				<origin xyz="-0.02 -0.015 0.0" rpy="1.5708 0.623 0.0" />
 				<parent link="support_top_link" />
 				<child link="camera_link_support_axis" />
@@ -87,5 +87,5 @@
 		</xacro:unless>
 		<sensor_imu parent="base_link" /> <!-- guardian_robot_control uses imu to update odometry -->
-		<sensor_hokuyo_front parent="base_link" prefix="front_laser" visualize="true" origin_x="0.46" origin_y="-0.0025" origin_z="0.2595" origin_roll="0.0" origin_pitch="0.0" origin_yaw="-0.026" />
+		<sensor_hokuyo_front parent="base_link" prefix="front_laser" visualize="true" origin_x="0.026" origin_y="-0.0015" origin_z="0.0565" origin_roll="-0.013" origin_pitch="0.0" origin_yaw="-0.023" />
 		<sensor_hokuyo_back parent="base_link" prefix="back_laser" visualize="true" origin_x="-0.433" origin_y="-0.0085" origin_z="0.3065" origin_roll="0.0" origin_pitch="0.0" origin_yaw="${PI}" />
 	</xacro:macro>

File: guardian_sim/guardian_description/urdf/sensors/hokuyo_front.urdf.xacro (robot description, xacro)
@@ -19,5 +19,5 @@
 		<joint name="hokuyo_${prefix}_tilt_support_joint" type="fixed">
 			<axis xyz="0 1 0" />
-			<origin xyz="${origin_x} ${origin_y} ${origin_z}" rpy="${origin_roll} ${origin_pitch} ${origin_yaw}" />
+			<origin xyz="0.46 -0.0025 0.2535" rpy="0.0 0.0 0.0" />
 			<parent link="${parent}" />
 			<child link="hokuyo_${prefix}_tilt_support_link" />
@@ -52,5 +52,5 @@
 		<joint name="hokuyo_${prefix}_joint" type="fixed">
 			<axis xyz="0 1 0" />
-			<origin xyz="0.026 -0.0015 0.0565" />
+			<origin xyz="${origin_x} ${origin_y} ${origin_z}" rpy="${origin_roll} ${origin_pitch} ${origin_yaw}" />
 			<parent link="hokuyo_${prefix}_tilt_axis_link" />
 			<child link="hokuyo_${prefix}_link" />

Commit message: Added arm description.

File: guardian_sim/guardian_description/urdf/guardian_base.urdf.xacro (robot description, xacro)
@@ -2,8 +2,14 @@
 <robot xmlns:xacro="http://www.ros.org/wiki/xacro">
 	<xacro:include filename="$(find guardian_description)/urdf/guardian_base.gazebo" />
-	<xacro:include filename="$(find guardian_description)/urdf/sensors/kinect.urdf.xacro"/>
+	<xacro:include filename="$(find guardian_description)/urdf/sensors/kinect.urdf.xacro" />
 	<xacro:include filename="$(find guardian_description)/urdf/sensors/imu.urdf.xacro" />
 	<xacro:include filename="$(find guardian_description)/urdf/sensors/hokuyo_front.urdf.xacro" />
 	<xacro:include filename="$(find guardian_description)/urdf/sensors/hokuyo_back.urdf.xacro" />
+	<!-- schunk arm dependencies -->
+	<xacro:include filename="$(find cob_description)/urdf/common.xacro" />
+	<xacro:include filename="$(find schunk_description)/urdf/materials.urdf.xacro" />
+	<xacro:include filename="$(find cob_description)/gazebo/gazebo.urdf.xacro" />
+	<xacro:include filename="$(find schunk_lwa4p)/calibration/calibration.urdf.xacro" />
+	<xacro:include filename="$(find schunk_description)/urdf/lwa4p/lwa4p.urdf.xacro" />
 	<xacro:macro name="guardian_base" params="base_footprint_z use_simulated_kinect">
 		<!-- BASE FOOTPRINT -->
@@ -38,10 +44,6 @@
 			<child link="support_top_link" />
 		</joint>
-		<!-- <link name="projector_link" />
-		<joint name="projector_joint" type="fixed">
-			<origin xyz="-0.07 0.031 -0.041" rpy="1.5707 0 0" />
-			<parent link="support_top_link" />
-			<child link="projector_link" />
-		</joint> -->
+		<!-- <link name="projector_link" /> <joint name="projector_joint" type="fixed"> <origin xyz="-0.07 0.031 -0.041" rpy="1.5707 0 0" /> <parent link="support_top_link"
+			/> <child link="projector_link" /> </joint> -->
 		<!-- BASE_LINK (Grey) -->
 		<link name="base_link"> <!-- center of wheels -> rotation axis -->
@@ -68,7 +70,111 @@
 			</collision>
 		</link>
+		<!-- SCHUNK LWA4P ARM -->
+		<xacro:schunk_lwa4p name="arm" parent="base_link">
+			<origin xyz="0.15 0 0.37" rpy="0 0 0" />
+		</xacro:schunk_lwa4p>
+		<!-- ft45 force and torque sensor -->
+		<link name="ft45_link">
+			<visual>
+				<origin xyz="0 0 -0.025" rpy="0 0 0" />
+				<geometry>
+					<cylinder radius="0.04" length="0.05" />
+				</geometry>
+			</visual>
+			<collision>
+				<origin xyz="0 0 -0.025" rpy="0 0 0" />
+				<geometry>
+					<cylinder radius="0.04" length="0.05" />
+				</geometry>
+			</collision>
+		</link>
+		<joint name="ft45_joint" type="fixed">
+			<parent link="arm_6_link" />
+			<child link="ft45_link" />
+			<origin xyz="0 0 0.13" rpy="0 0 0" />
+		</joint>
+		<!-- camera coupler -->
+		<link name="coupler_link">
+			<visual>
+				<origin xyz="0 0 -0.002" rpy="0 0 0" />
+				<geometry>
+					<box size="0.24 0.1 0.002" />
+				</geometry>
+			</visual>
+			<collision>
+				<origin xyz="0 0 -0.002" rpy="0 0 0" />
+				<geometry>
+					<box size="0.24 0.1 0.002" />
+				</geometry>
+			</collision>
+		</link>
+		<joint name="coupler_joint" type="fixed">
+			<parent link="ft45_link" />
+			<child link="coupler_link" />
+			<origin xyz="0 0 0.002" rpy="0 0 0" />
+		</joint>
+		<!-- camera -->
+		<link name="v_camera_link">
+			<visual>
+				<origin xyz="0 0 -0.01" rpy="0 0 0" />
+				<geometry>
+					<box size="0.03 0.07 0.02" />
+				</geometry>
+			</visual>
+			<collision>
+				<origin xyz="0 0 -0.01" rpy="0 0 0" />
+				<geometry>
+					<box size="0.03 0.07 0.02" />
+				</geometry>
+			</collision>
+		</link>
+		<joint name="v_camera_joint" type="fixed">
+			<parent link="coupler_link" />
+			<child link="v_camera_link" />
+			<origin xyz="-0.095 0 0.02" rpy="0 0 0" />
+		</joint>
+		<!-- projector -->
+		<link name="projector_link">
+			<visual>
+				<origin xyz="0 0 -0.05" rpy="0 0 0" />
+				<geometry>
+					<box size="0.05 0.15 0.1" />
+				</geometry>
+			</visual>
+			<collision>
+				<origin xyz="0 0 -0.05" rpy="0 0 0" />
+				<geometry>
+					<box size="0.05 0.15 0.1" />
+				</geometry>
+			</collision>
+		</link>
+		<joint name="projector_joint" type="fixed">
+			<parent link="coupler_link" />
+			<child link="projector_link" />
+			<origin xyz="0.08 0 0.02" rpy="0 0 0" />
+		</joint>
+		<!-- welding tool -->
+		<link name="tool_link">
+			<visual>
+				<origin xyz="0 0 -0.07" rpy="0 0 0" />
+				<geometry>
+					<cylinder radius="0.03" length="0.14" />
+				</geometry>
+			</visual>
+			<collision>
+				<origin xyz="0 0 -0.07" rpy="0 0 0" />
+				<geometry>
+					<cylinder radius="0.03" length="0.14" />
+				</geometry>
+			</collision>
+		</link>
+		<joint name="tool_joint" type="fixed">
+			<parent link="coupler_link" />
+			<child link="tool_link" />
+			<origin xyz="0 0 0.14" rpy="0 0 0" />
+		</joint>
 		<!-- ################# SENSORS ################# -->
 		<xacro:if value="${use_simulated_kinect}">
- 			<sensor_kinect parent="base_link"/>
+			<sensor_kinect parent="base_link" />
 		</xacro:if>
 		<xacro:unless value="${use_simulated_kinect}">
@@ -87,6 +193,8 @@
 		</xacro:unless>
 		<sensor_imu parent="base_link" /> <!-- guardian_robot_control uses imu to update odometry -->
-		<sensor_hokuyo_front parent="base_link" prefix="front_laser" visualize="true" origin_x="0.026" origin_y="-0.0015" origin_z="0.0565" origin_roll="-0.013" origin_pitch="0.0" origin_yaw="-0.023" />
-		<sensor_hokuyo_back parent="base_link" prefix="back_laser" visualize="true" origin_x="-0.433" origin_y="-0.0085" origin_z="0.3065" origin_roll="0.0" origin_pitch="0.0" origin_yaw="${PI}" />
+		<sensor_hokuyo_front parent="base_link" prefix="front_laser" visualize="true" origin_x="0.026" origin_y="-0.0015" origin_z="0.0565"
+			origin_roll="-0.013" origin_pitch="0.0" origin_yaw="-0.023" />
+		<sensor_hokuyo_back parent="base_link" prefix="back_laser" visualize="true" origin_x="-0.433" origin_y="-0.0085" origin_z="0.3065"
+			origin_roll="0.0" origin_pitch="0.0" origin_yaw="${PI}" />
 	</xacro:macro>
 </robot>

Commit message: Moved schunk arm xacro elements to separate file.

File: guardian_sim/guardian_description/urdf/guardian_base.urdf.xacro (robot description, xacro)
@@ -2,15 +2,8 @@
 <robot xmlns:xacro="http://www.ros.org/wiki/xacro">
 	<xacro:include filename="$(find guardian_description)/urdf/guardian_base.gazebo" />
-	<xacro:include filename="$(find guardian_description)/urdf/sensors/kinect.urdf.xacro" />
 	<xacro:include filename="$(find guardian_description)/urdf/sensors/imu.urdf.xacro" />
 	<xacro:include filename="$(find guardian_description)/urdf/sensors/hokuyo_front.urdf.xacro" />
 	<xacro:include filename="$(find guardian_description)/urdf/sensors/hokuyo_back.urdf.xacro" />
-	<!-- schunk arm dependencies -->
-	<xacro:include filename="$(find cob_description)/urdf/common.xacro" />
-	<xacro:include filename="$(find schunk_description)/urdf/materials.urdf.xacro" />
-	<xacro:include filename="$(find cob_description)/gazebo/gazebo.urdf.xacro" />
-	<xacro:include filename="$(find schunk_lwa4p)/calibration/calibration.urdf.xacro" />
-	<xacro:include filename="$(find schunk_description)/urdf/lwa4p/lwa4p.urdf.xacro" />
-	<xacro:macro name="guardian_base" params="base_footprint_z use_simulated_kinect">
+	<xacro:macro name="guardian_base" params="base_footprint_z use_simulated_kinect use_schunk_arm" >
 		<!-- BASE FOOTPRINT -->
 		<!-- base_footprint is a fictitious link(frame) that is on the ground right below base_link origin, navigation stack depends on this frame -->
@@ -70,110 +63,12 @@
 			</collision>
 		</link>
-		<!-- SCHUNK LWA4P ARM -->
-		<xacro:schunk_lwa4p name="arm" parent="base_link">
-			<origin xyz="0.15 0 0.37" rpy="0 0 0" />
-		</xacro:schunk_lwa4p>
-		<!-- ft45 force and torque sensor -->
-		<link name="ft45_link">
-			<visual>
-				<origin xyz="0 0 -0.025" rpy="0 0 0" />
-				<geometry>
-					<cylinder radius="0.04" length="0.05" />
-				</geometry>
-			</visual>
-			<collision>
-				<origin xyz="0 0 -0.025" rpy="0 0 0" />
-				<geometry>
-					<cylinder radius="0.04" length="0.05" />
-				</geometry>
-			</collision>
-		</link>
-		<joint name="ft45_joint" type="fixed">
-			<parent link="arm_6_link" />
-			<child link="ft45_link" />
-			<origin xyz="0 0 0.13" rpy="0 0 0" />
-		</joint>
-		<!-- camera coupler -->
-		<link name="coupler_link">
-			<visual>
-				<origin xyz="0 0 -0.002" rpy="0 0 0" />
-				<geometry>
-					<box size="0.24 0.1 0.002" />
-				</geometry>
-			</visual>
-			<collision>
-				<origin xyz="0 0 -0.002" rpy="0 0 0" />
-				<geometry>
-					<box size="0.24 0.1 0.002" />
-				</geometry>
-			</collision>
-		</link>
-		<joint name="coupler_joint" type="fixed">
-			<parent link="ft45_link" />
-			<child link="coupler_link" />
-			<origin xyz="0 0 0.002" rpy="0 0 0" />
-		</joint>
-		<!-- camera -->
-		<link name="v_camera_link">
-			<visual>
-				<origin xyz="0 0 -0.01" rpy="0 0 0" />
-				<geometry>
-					<box size="0.03 0.07 0.02" />
-				</geometry>
-			</visual>
-			<collision>
-				<origin xyz="0 0 -0.01" rpy="0 0 0" />
-				<geometry>
-					<box size="0.03 0.07 0.02" />
-				</geometry>
-			</collision>
-		</link>
-		<joint name="v_camera_joint" type="fixed">
-			<parent link="coupler_link" />
-			<child link="v_camera_link" />
-			<origin xyz="-0.095 0 0.02" rpy="0 0 0" />
-		</joint>
-		<!-- projector -->
-		<link name="projector_link">
-			<visual>
-				<origin xyz="0 0 -0.05" rpy="0 0 0" />
-				<geometry>
-					<box size="0.05 0.15 0.1" />
-				</geometry>
-			</visual>
-			<collision>
-				<origin xyz="0 0 -0.05" rpy="0 0 0" />
-				<geometry>
-					<box size="0.05 0.15 0.1" />
-				</geometry>
-			</collision>
-		</link>
-		<joint name="projector_joint" type="fixed">
-			<parent link="coupler_link" />
-			<child link="projector_link" />
-			<origin xyz="0.08 0 0.02" rpy="0 0 0" />
-		</joint>
-		<!-- welding tool -->
-		<link name="tool_link">
-			<visual>
-				<origin xyz="0 0 -0.07" rpy="0 0 0" />
-				<geometry>
-					<cylinder radius="0.03" length="0.14" />
-				</geometry>
-			</visual>
-			<collision>
-				<origin xyz="0 0 -0.07" rpy="0 0 0" />
-				<geometry>
-					<cylinder radius="0.03" length="0.14" />
-				</geometry>
-			</collision>
-		</link>
-		<joint name="tool_joint" type="fixed">
-			<parent link="coupler_link" />
-			<child link="tool_link" />
-			<origin xyz="0 0 0.14" rpy="0 0 0" />
-		</joint>
+		<!-- ################# ARM ################# -->
+		<!-- <xacro:if value="${use_schunk_arm}">
+			<xacro:include filename="$(find guardian_description)/urdf/schunk_arm.urdf.xacro" />
+			<schunk_arm parent="base_link" />
+		</xacro:if> -->
 		<!-- ################# SENSORS ################# -->
 		<xacro:if value="${use_simulated_kinect}">
+			<xacro:include filename="$(find guardian_description)/urdf/sensors/kinect.urdf.xacro" />
 			<sensor_kinect parent="base_link" />
 		</xacro:if>

File: guardian_sim/guardian_description/urdf/guardian_tracks.urdf.xacro (robot description, xacro)
@@ -5,5 +5,5 @@
 	<xacro:include filename="$(find guardian_description)/urdf/track_wheel.urdf.xacro" />
 	<!-- ###### BASE ###### -->
-	<guardian_base base_footprint_z="0.0635" use_simulated_kinect="false" />
+	<guardian_base base_footprint_z="0.0635" use_simulated_kinect="false" use_schunk_arm="false" />
 	<!-- ###### TRACKS ###### -->
 	<!-- visual -->

File: guardian_sim/guardian_description/urdf/guardian_wheels.urdf.xacro (robot description, xacro)
@@ -7,5 +7,5 @@
 	<xacro:include filename="$(find guardian_description)/urdf/wheel.urdf.xacro" />
 	<!-- ###### BASE ###### -->
-	<guardian_base base_footprint_z="0.175" use_simulated_kinect="false" /> <!-- wheels radius -->
+	<guardian_base base_footprint_z="0.175" use_simulated_kinect="false" use_schunk_arm="false" /> <!-- wheels radius -->
 	<!-- ###### TRACKS ###### -->
 	<track parent="base_link" prefix="left_track" joint_yaw="${PI}" />

File: guardian_sim/guardian_description/urdf/sensors/kinect.urdf.xacro (robot description, xacro)
@@ -4,5 +4,5 @@
   <xacro:include filename="$(find guardian_description)/urdf/sensors/kinect_gazebo.urdf.xacro"/>
   <!-- Parameterised in part by the values in turtlebot_properties.urdf.xacro -->
-  <xacro:macro name="sensor_kinect" params="parent">
+  <xacro:macro name="sensor_kinect" params="parent" >
     <joint name="camera_rgb_joint" type="fixed">
       <origin xyz="${cam_px} ${cam_py} ${cam_pz}" rpy="${cam_or} ${cam_op} ${cam_oy}"/>

Commit message: Improved laser calibration.

File: guardian_sim/guardian_description/urdf/guardian_base.urdf.xacro (robot description, xacro)
@@ -88,6 +88,9 @@
 		</xacro:unless>
 		<sensor_imu parent="base_link" /> <!-- guardian_robot_control uses imu to update odometry -->
-		<sensor_hokuyo_front parent="base_link" prefix="front_laser" visualize="true" origin_x="0.03" origin_y="0.005" origin_z="0.0565" origin_roll="-0.013" origin_pitch="0.0" origin_yaw="0.013" />
-		<sensor_hokuyo_back parent="base_link" prefix="back_laser" visualize="true" origin_x="-0.433" origin_y="-0.0085" origin_z="0.3065" origin_roll="0.0" origin_pitch="0.0" origin_yaw="${PI}" />
+		<sensor_hokuyo_front parent="base_link" prefix="front_laser" visualize="true"
+			support_x="0.4625" 	support_y="-0.0025" 	support_z="0.2535" 		support_roll="0.0" 		support_pitch="0.0" 	support_yaw="0.0"
+			sensor_x ="0.03" 	sensor_y="0.005" 		sensor_z ="0.0565" 		sensor_roll ="-0.013" 	sensor_pitch ="0.0" 	sensor_yaw ="0.013" />
+		<sensor_hokuyo_back 	parent="base_link" 		prefix="back_laser" 	visualize="true"
+			origin_x ="-0.431" 	origin_y="-0.0085" 		origin_z ="0.3065" 		origin_roll ="0.10" 	origin_pitch ="0.0" 	origin_yaw ="${PI}" />
 	</xacro:macro>
 </robot>

File: guardian_sim/guardian_description/urdf/sensors/hokuyo_front.urdf.xacro (robot description, xacro)
@@ -8,5 +8,5 @@
 	<xacro:property name="ptz_joint_damping" value="0.1" />
 	<xacro:property name="ptz_mechanical_reduction" value="1.0" />
-	<xacro:macro name="sensor_hokuyo_front" params="parent prefix visualize origin_x origin_y origin_z origin_roll origin_pitch origin_yaw"> <!-- origin -> laser rotation axis center -->
+	<xacro:macro name="sensor_hokuyo_front" params="parent prefix visualize support_x support_y support_z support_roll support_pitch support_yaw sensor_x sensor_y sensor_z sensor_roll sensor_pitch sensor_yaw"> <!-- sensor -> laser rotation axis center -->
 		<!-- front laser tilting platform -->
 		<link name="hokuyo_${prefix}_tilt_support_link" >
@@ -19,5 +19,5 @@
 		<joint name="hokuyo_${prefix}_tilt_support_joint" type="fixed">
 			<axis xyz="0 1 0" />
-			<origin xyz="0.46 -0.0025 0.2535" rpy="0.0 0.0 0.0" />
+			<origin xyz="${support_x} ${support_y} ${support_z}" rpy="${support_roll} ${support_pitch} ${support_yaw}" />
 			<parent link="${parent}" />
 			<child link="hokuyo_${prefix}_tilt_support_link" />
@@ -54,5 +54,5 @@
 		<joint name="hokuyo_${prefix}_joint" type="fixed">
 			<axis xyz="0 1 0" />
-			<origin xyz="${origin_x} ${origin_y} ${origin_z}" rpy="${origin_roll} ${origin_pitch} ${origin_yaw}" />
+			<origin xyz="${sensor_x} ${sensor_y} ${sensor_z}" rpy="${sensor_roll} ${sensor_pitch} ${sensor_yaw}" />
 			<parent link="hokuyo_${prefix}_tilt_axis_link" />
 			<child link="hokuyo_${prefix}_link" />
