Commit message: Improved arm integration with robot platform.

File: guardian_sim/guardian_description/urdf/guardian_base.urdf.xacro (robot description, xacro)
@@ -6,4 +6,5 @@
 	<xacro:include filename="$(find guardian_description)/urdf/sensors/hokuyo_back.urdf.xacro" />
 	<xacro:include filename="$(find guardian_description)/urdf/sensors/kinect.urdf.xacro" />
+	<xacro:include filename="$(find guardian_description)/urdf/schunk_arm.urdf.xacro" />
 	<xacro:macro name="guardian_base" params="base_footprint_z use_simulated_kinect use_schunk_arm" >
 		<!-- BASE FOOTPRINT -->
@@ -65,8 +66,20 @@
 		</link>
 		<!-- ################# ARM ################# -->
-		<!-- <xacro:if value="${use_schunk_arm}">
-			<xacro:include filename="$(find guardian_description)/urdf/schunk_arm.urdf.xacro" />
-			<schunk_arm parent="base_link" />
-		</xacro:if> -->
+		<link name="arm_link">
+			<visual>
+				<origin xyz="0 0 0" rpy="0 0 0" />
+				<geometry>
+					<cylinder radius="0.001" length="0.001" />
+				</geometry>
+			</visual>
+		</link>
+		<joint name="arm_joint" type="fixed">
+			<parent link="base_link" />
+			<child link="arm_link" />
+			<origin xyz="0.15 0 -0.13" rpy="0 0 0" />
+		</joint>
+		<xacro:if value="${use_schunk_arm}">
+			<schunk_arm parent="arm_link" />
+		</xacro:if>
 		<!-- ################# SENSORS ################# -->
 		<xacro:if value="${use_simulated_kinect}">

File: guardian_sim/guardian_description/urdf/guardian_tracks.urdf.xacro (robot description, xacro)
@@ -5,5 +5,5 @@
 	<xacro:include filename="$(find guardian_description)/urdf/track_wheel.urdf.xacro" />
 	<!-- ###### BASE ###### -->
-	<guardian_base base_footprint_z="0.0635" use_simulated_kinect="$(arg useSimulatedKinect)" use_schunk_arm="false" />
+	<guardian_base base_footprint_z="0.0635" use_simulated_kinect="$(arg useSimulatedKinect)" use_schunk_arm="true" />
 	<!-- ###### TRACKS ###### -->
 	<!-- visual -->

File: guardian_sim/guardian_description/urdf/schunk_arm.urdf.xacro (robot description, xacro)
@@ -1,4 +1,4 @@
 <?xml version="1.0"?>
-<robot name="schunk_arm"  xmlns:xacro="http://ros.org/wiki/xacro">
+<robot xmlns:xacro="http://ros.org/wiki/xacro">
 	<!-- schunk arm dependencies -->
 	<xacro:include filename="$(find cob_description)/urdf/common.xacro" />
@@ -10,5 +10,5 @@
 		<!-- SCHUNK LWA4P ARM -->
 		<xacro:schunk_lwa4p name="arm" parent="${parent}">
-			<origin xyz="0.15 0 0.37" rpy="0 0 0" />
+			<origin xyz="0.0 0 0.5" rpy="0 0 0" />
 		</xacro:schunk_lwa4p>
 		<!-- ft45 force and torque sensor -->
@@ -73,5 +73,5 @@
 		</joint>
 		<!-- projector -->
-		<link name="projector_link">
+		<!-- <link name="projector_link">
 			<visual>
 				<origin xyz="0 0 -0.05" rpy="0 0 0" />
@@ -91,5 +91,5 @@
 			<child link="projector_link" />
 			<origin xyz="0.08 0 0.02" rpy="0 0 0" />
-		</joint>
+		</joint> -->
 		<!-- welding tool -->
 		<link name="tool_link">

Commit message: Fixed camera and projector TFs.

File: guardian_sim/guardian_description/urdf/guardian_base.urdf.xacro (robot description, xacro)
@@ -77,5 +77,5 @@
 			<parent link="base_link" />
 			<child link="arm_link" />
-			<origin xyz="0.15 0 -0.13" rpy="0 0 0" />
+			<origin xyz="0.15 0 -0.15" rpy="0 0 0" />
 		</joint>
 		<xacro:if value="${use_schunk_arm}">

File: guardian_sim/guardian_description/urdf/schunk_arm.urdf.xacro (robot description, xacro)
@@ -67,13 +67,13 @@
 		  </collision>
 		</link>
-		<!--joint name="v_camera_joint" type="fixed">
+		<joint name="v_camera_joint" type="fixed">
 			<parent link="coupler_link" />
 			<child link="v_camera_link" />
 			<origin xyz="-0.11 0 0" rpy="0 0 1.5708" />
-		</joint-->
+		</joint>
 		<!-- projector -->
 		<link name="projector_link">
 		  <visual>
-		    <origin xyz="0.05 0 -0.05" rpy="0 0 0" />
+		    <origin xyz="0.150 0 -0.05" rpy="0 0 0" />
 		    <geometry>
 		      <box size="0.155 0.04 0.1" />
@@ -81,5 +81,5 @@
 		  </visual>
 		  <collision>
-		    <origin xyz="0.05 0 -0.05" rpy="0 0 0" />
+		    <origin xyz="0.150 0 -0.05" rpy="0 0 0" />
 		    <geometry>
 		      <box size="0.155 0.04 0.1" />
@@ -87,13 +87,18 @@
 		  </collision>
 		</link>
-		<joint name="projector_joint" type="fixed">
-		  <parent link="coupler_link" />
-		  <child link="projector_link" />
-		  <origin xyz="0.05 -0.075 0.02" rpy="0 0 0" />
-		</joint>
-		<joint name="v_camera_joint" type="fixed">
+		<!--joint name="v_camera_joint" type="fixed">
 		  <parent link="projector_link" />
 		  <child link="v_camera_link" />
 		  <origin xyz="-0.227186 0.0744 -0.0052" rpy="0.00322 0.02632 1.56316" />
+		</joint-->
+		<!--joint name="projector_joint" type="fixed">
+		  <parent link="v_camera_link" />
+		  <child link="projector_link" />
+		  <origin xyz="-0.227186 0.0744 -0.0052" rpy="0.00322 0.02632 1.56316" />
+		</joint-->
+		<joint name="projector_joint" type="fixed">
+		  <parent link="v_camera_link" />
+		  <child link="projector_link" />
+		  <origin xyz="-0.076 -0.247 0.045" rpy="-0.026 0.003 -1.56316" />
 		</joint>
 		<!-- welding tool -->

Commit message: Added option to use planar lasers in simulation. Added gpu support for gazebo lasers. Changed kinect pose to point to the ceiling. Increased laser tilt range.

File: guardian_sim/guardian_description/urdf/guardian_base.urdf.xacro (robot description, xacro)
@@ -7,5 +7,5 @@
 	<xacro:include filename="$(find guardian_description)/urdf/sensors/kinect.urdf.xacro" />
 	<xacro:include filename="$(find guardian_description)/urdf/schunk_arm.urdf.xacro" />
-	<xacro:macro name="guardian_base" params="base_footprint_z use_simulated_kinect use_schunk_arm" >
+	<xacro:macro name="guardian_base" params="base_footprint_z use_simulated_kinect use_schunk_arm use_planar_lasers" >
 		<!-- BASE FOOTPRINT -->
 		<!-- base_footprint is a fictitious link(frame) that is on the ground right below base_link origin, navigation stack depends on this frame -->
@@ -101,9 +101,18 @@
 		</xacro:unless>
 		<sensor_imu parent="base_link" /> <!-- guardian_robot_control uses imu to update odometry -->
-		<sensor_hokuyo_front parent="base_link" prefix="front_laser" visualize="true"
-			support_x="0.46" 	support_y="0.0" 		support_z="0.2535" 		support_roll="0.0" 		support_pitch="0.0" 	support_yaw="0.0"
-			sensor_x ="0.03" 	sensor_y="0.0" 		sensor_z ="0.0735" 		sensor_roll ="-0.05" 		sensor_pitch ="0.0" 	sensor_yaw ="0.0" />
-		<sensor_hokuyo_back 	parent="base_link" 		prefix="back_laser" 	visualize="true"
-			origin_x ="-0.43" 	origin_y="-0.0045" 		origin_z ="0.3435" 		origin_roll ="0.12" 	origin_pitch ="0.0" 	origin_yaw ="${PI-0.015}" />
+		<xacro:if value="${use_planar_lasers}">
+			<sensor_hokuyo_front parent="base_link" prefix="front_laser" visualize="true"
+				support_x="0.46" 	support_y="0.0" 		support_z="0.2535" 		support_roll="0.0" 		support_pitch="0.0" 	support_yaw="0.0"
+				sensor_x ="0.03" 	sensor_y="0.0" 			sensor_z ="0.0735" 		sensor_roll ="0" 		sensor_pitch ="0.0" 	sensor_yaw ="0.0" />
+			<sensor_hokuyo_back 	parent="base_link" 		prefix="back_laser" 	visualize="true"
+				origin_x ="-0.43" 	origin_y="-0.0045" 		origin_z ="0.3435" 		origin_roll ="0" 		origin_pitch ="0.0" 	origin_yaw ="${PI}" />
+		</xacro:if>
+		<xacro:unless value="${use_planar_lasers}">
+			<sensor_hokuyo_front parent="base_link" prefix="front_laser" visualize="true"
+				support_x="0.46" 	support_y="0.0" 		support_z="0.2535" 		support_roll="0.0" 		support_pitch="0.0" 	support_yaw="0.0"
+				sensor_x ="0.03" 	sensor_y="0.0" 			sensor_z ="0.0735" 		sensor_roll ="-0.05" 	sensor_pitch ="0.0" 	sensor_yaw ="0.0" />
+			<sensor_hokuyo_back 	parent="base_link" 		prefix="back_laser" 	visualize="true"
+				origin_x ="-0.43" 	origin_y="-0.0045" 		origin_z ="0.3435" 		origin_roll ="0.12" 	origin_pitch ="0.0" 	origin_yaw ="${PI-0.015}" />
+		</xacro:unless>
 	</xacro:macro>
 </robot>

File: guardian_sim/guardian_description/urdf/guardian_tracks.urdf.xacro (robot description, xacro)
@@ -6,5 +6,5 @@
 	<!-- args: useSimulatedKinect useSchunkArm publishOdometryTf publishOdometryMsg -->
 	<!-- ###### BASE ###### -->
-	<guardian_base base_footprint_z="0.0635" use_simulated_kinect="$(arg useSimulatedKinect)" use_schunk_arm="$(arg useSchunkArm)" />
+	<guardian_base base_footprint_z="0.0635" use_simulated_kinect="$(arg useSimulatedKinect)" use_schunk_arm="$(arg useSchunkArm)" use_planar_lasers="$(arg usePlanarLasers) />
 	<!-- ###### TRACKS ###### -->
 	<!-- visual -->

File: guardian_sim/guardian_description/urdf/guardian_wheels.urdf.xacro (robot description, xacro)
@@ -8,5 +8,5 @@
 	<!-- args: useSimulatedKinect useSchunkArm -->
 	<!-- ###### BASE ###### -->
-	<guardian_base base_footprint_z="0.175" use_simulated_kinect="$(arg useSimulatedKinect)" use_schunk_arm="$(arg useSchunkArm)" /> <!-- wheels radius -->
+	<guardian_base base_footprint_z="0.175" use_simulated_kinect="$(arg useSimulatedKinect)" use_schunk_arm="$(arg useSchunkArm)" use_planar_lasers="$(arg usePlanarLasers)" /> <!-- wheels radius -->
 	<!-- ###### TRACKS ###### -->
 	<track parent="base_link" prefix="left_track" joint_yaw="${PI}" />

File: guardian_sim/guardian_description/urdf/sensors/hokuyo_back.urdf.xacro (robot description, xacro)
@@ -28,5 +28,5 @@
 		<gazebo reference="hokuyo_${prefix}_link">
 			<material>Gazebo/FlatBlack</material>
-			<sensor type="ray" name="${prefix}_sensor">
+			<sensor type="gpu_ray" name="${prefix}_sensor">
 				<pose>0 0 0 0 0 0</pose>
 				<visualize>${visualize}</visualize>
@@ -53,5 +53,5 @@
 					</noise>
 				</ray>
-				<plugin name="${prefix}_plugin" filename="libgazebo_ros_laser_2D.so">
+				<plugin name="${prefix}_plugin" filename="libgazebo_ros_gpu_laser.so">
 					<topicName>/guardian/laser_horizontal_back</topicName>
 					<frameName>hokuyo_${prefix}_link</frameName>

File: guardian_sim/guardian_description/urdf/sensors/hokuyo_front.urdf.xacro (robot description, xacro)
@@ -68,5 +68,5 @@
 		<gazebo reference="hokuyo_${prefix}_link">
 			<material>Gazebo/Grey</material>
-			<sensor type="ray" name="${prefix}_sensor">
+			<sensor type="gpu_ray" name="${prefix}_sensor">
 				<pose>0 0 0 0 0 0</pose>
 				<visualize>${visualize}</visualize>
@@ -92,5 +92,5 @@
 					</noise>
 				</ray>
-				<plugin name="${prefix}_plugin" filename="libgazebo_ros_laser_2D.so">
+				<plugin name="${prefix}_plugin" filename="libgazebo_ros_gpu_laser.so">
 					<topicName>/guardian/laser_tilt_front</topicName>
 					<frameName>hokuyo_${prefix}_link</frameName>

File: guardian_sim/guardian_description/urdf/sensors/kinect_gazebo.urdf.xacro (robot description, xacro)
@@ -17,5 +17,5 @@
           <clip>
             <near>0.8</near> <!-- specs -> 0.8 -->
-            <far>4.0</far> <!-- specs -> 4.0 -->
+            <far>5.0</far> <!-- specs -> 4.0 -->
           </clip>
         </camera>
@@ -23,5 +23,5 @@
           <cameraName>camera</cameraName>
           <alwaysOn>true</alwaysOn>
-          <updateRate>30.0</updateRate> <!-- specs -> 30 -->
+          <updateRate>10.0</updateRate> <!-- specs -> 30 -->
           <imageTopicName>rgb/image_raw</imageTopicName>
           <depthImageTopicName>depth/image_raw</depthImageTopicName>
@@ -37,4 +37,5 @@
           <distortion_t2>0.0</distortion_t2>
           <pointCloudCutoff>0.8</pointCloudCutoff> <!-- specs -> 0.8 -->
+          <pointCloudCutoffMax>5.0</pointCloudCutoffMax>
         </plugin>
       </sensor>

File: guardian_sim/guardian_description/urdf/sensors/kinect_properties.urdf.xacro (robot description, xacro)
@@ -2,9 +2,9 @@
 <robot>
 	<property name="M_PI" value="3.1415926535897931" />
-	<property name="cam_px" value="0.306" />
+	<property name="cam_px" value="0.326" />
 	<property name="cam_py" value="0" />
-	<property name="cam_pz" value="0.423" />
-	<property name="cam_or" value="0" />
-	<property name="cam_op" value="-0.78539816339" />
-	<property name="cam_oy" value="0" />
+	<property name="cam_pz" value="0.385" />
+	<property name="cam_or" value="1.5707" />
+	<property name="cam_op" value="-0.261799" />
+	<property name="cam_oy" value="0.349066" />
 </robot>

Commit message: Configurations for colrobot van tests.

File: guardian_sim/guardian_description/urdf/guardian_base.urdf.xacro (robot description, xacro)
@@ -11,10 +11,10 @@
 		<!-- base_footprint is a fictitious link(frame) that is on the ground right below base_link origin, navigation stack depends on this frame -->
 		<link name="base_footprint">
-			<visual>
-				<origin xyz="0 0 0" rpy="0 0 0" />
-				<geometry>
-					<box size="0.005 0.005 0.005" />
-				</geometry>
-			</visual>
+<!-- 			<visual> -->
+<!-- 				<origin xyz="0 0 0" rpy="0 0 0" /> -->
+<!-- 				<geometry> -->
+<!-- 					<box size="0.005 0.005 0.005" /> -->
+<!-- 				</geometry> -->
+<!-- 			</visual> -->
 		</link>
 		<joint name="base_footprint_joint" type="fixed">
@@ -57,11 +57,11 @@
 				</material>
 			</visual>
-			<collision>
-				<origin xyz="0 0 0.08" rpy="0 0 0 " />
-				<geometry>
+<!-- 			<collision> -->
+<!-- 				<origin xyz="0 0 0.08" rpy="0 0 0 " /> -->
+<!-- 				<geometry> -->
 					<!-- <box size = "1.127 0.497 0.28"/> --> <!-- includes tracks, making it just tall enough not to hit the laser beams -->
-					<box size="1.127 0.497 0.25" /> <!-- this is not enough -->
-				</geometry>
-			</collision>
+<!-- 					<box size="1.127 0.497 0.25" /> this is not enough -->
+<!-- 				</geometry> -->
+<!-- 			</collision> -->
 		</link>
 		<!-- ################# ARM ################# -->
@@ -102,15 +102,15 @@
 		<sensor_imu parent="base_link" /> <!-- guardian_robot_control uses imu to update odometry -->
 		<xacro:if value="${use_planar_lasers}">
-			<sensor_hokuyo_front parent="base_link" prefix="front_laser" visualize="true"
+			<sensor_hokuyo_front parent="base_link" prefix="front_laser" visualize="false"
 				support_x="0.46" 	support_y="0.0" 		support_z="0.2535" 		support_roll="0.0" 		support_pitch="0.0" 	support_yaw="0.0"
 				sensor_x ="0.03" 	sensor_y="0.0" 			sensor_z ="0.0735" 		sensor_roll ="0" 		sensor_pitch ="0.0" 	sensor_yaw ="0.0" />
-			<sensor_hokuyo_back 	parent="base_link" 		prefix="back_laser" 	visualize="true"
+			<sensor_hokuyo_back 	parent="base_link" 		prefix="back_laser" 	visualize="false"
 				origin_x ="-0.43" 	origin_y="-0.0045" 		origin_z ="0.3435" 		origin_roll ="0" 		origin_pitch ="0.0" 	origin_yaw ="${PI}" />
 		</xacro:if>
 		<xacro:unless value="${use_planar_lasers}">
-			<sensor_hokuyo_front parent="base_link" prefix="front_laser" visualize="true"
+			<sensor_hokuyo_front parent="base_link" prefix="front_laser" visualize="false"
 				support_x="0.46" 	support_y="0.0" 		support_z="0.2535" 		support_roll="0.0" 		support_pitch="0.0" 	support_yaw="0.0"
 				sensor_x ="0.03" 	sensor_y="0.0" 			sensor_z ="0.0735" 		sensor_roll ="-0.05" 	sensor_pitch ="0.0" 	sensor_yaw ="0.0" />
-			<sensor_hokuyo_back 	parent="base_link" 		prefix="back_laser" 	visualize="true"
+			<sensor_hokuyo_back 	parent="base_link" 		prefix="back_laser" 	visualize="false"
 				origin_x ="-0.43" 	origin_y="-0.0045" 		origin_z ="0.3435" 		origin_roll ="0.12" 	origin_pitch ="0.0" 	origin_yaw ="${PI-0.015}" />
 		</xacro:unless>

File: guardian_sim/guardian_description/urdf/guardian_wheels.urdf.xacro (robot description, xacro)
@@ -14,6 +14,6 @@
 	<!-- track doesn't have collision, but the chassis has a collision bounding box -->
 	<!-- ###### WHEELS ###### -->
-	<wheel parent="base_link" prefix="back_left" origin_yaw="${PI}" reflect_link_y="-1" reflect_joint_x="-1" reflect_joint_y="1" material="Gazebo/FlatBlack" />
-	<wheel parent="base_link" prefix="back_right" origin_yaw="0" reflect_link_y="1" reflect_joint_x="-1" reflect_joint_y="-1" material="Gazebo/FlatBlack" />
+	<wheel parent="base_link" prefix="back_left" origin_yaw="${PI}" reflect_link_y="-1" reflect_joint_x="-1" reflect_joint_y="1" material="Gazebo/DarkGrey" />
+	<wheel parent="base_link" prefix="back_right" origin_yaw="0" reflect_link_y="1" reflect_joint_x="-1" reflect_joint_y="-1" material="Gazebo/DarkGrey" />
 	<wheel parent="base_link" prefix="front_left" origin_yaw="${PI}" reflect_link_y="-1" reflect_joint_x="1" reflect_joint_y="1" material="Gazebo/DarkGrey" />
 	<wheel parent="base_link" prefix="front_right" origin_yaw="0" reflect_link_y="1" reflect_joint_x="1" reflect_joint_y="-1" material="Gazebo/DarkGrey" />

File: guardian_sim/guardian_description/urdf/sensors/kinect_gazebo.urdf.xacro (robot description, xacro)
@@ -6,5 +6,5 @@
       <sensor type="depth" name="camera">
         <always_on>true</always_on>
-        <update_rate>30.0</update_rate> <!-- specs -> 30 -->
+        <update_rate>10.0</update_rate> <!-- specs -> 30 -->
         <camera>
           <horizontal_fov>${43*M_PI/180.0}</horizontal_fov> <!-- specs: 43.0*M_PI/180.0 -->
@@ -17,5 +17,5 @@
           <clip>
             <near>0.8</near> <!-- specs -> 0.8 -->
-            <far>5.0</far> <!-- specs -> 4.0 -->
+            <far>6.0</far> <!-- specs -> 4.0 -->
           </clip>
         </camera>
@@ -37,5 +37,5 @@
           <distortion_t2>0.0</distortion_t2>
           <pointCloudCutoff>0.8</pointCloudCutoff> <!-- specs -> 0.8 -->
-          <pointCloudCutoffMax>5.0</pointCloudCutoffMax>
+          <pointCloudCutoffMax>6.0</pointCloudCutoffMax>
         </plugin>
       </sensor>

File: guardian_sim/guardian_description/urdf/sensors/kinect_properties.urdf.xacro (robot description, xacro)
@@ -2,9 +2,10 @@
 <robot>
 	<property name="M_PI" value="3.1415926535897931" />
-	<property name="cam_px" value="0.326" />
+	<property name="cam_px" value="0.4" />
 	<property name="cam_py" value="0" />
-	<property name="cam_pz" value="0.385" />
-	<property name="cam_or" value="1.5707" />
-	<property name="cam_op" value="-0.261799" />
-	<property name="cam_oy" value="0.349066" />
+	<property name="cam_pz" value="0.33" />
+	<property name="cam_or" value="-1.5707" />
+	<property name="cam_op" value="0.0" />
+	<property name="cam_oy" value="0.1" />
+<!-- 	<property name="cam_oy" value="-0.42" /> -->
 </robot>

File: guardian_sim/guardian_description/urdf/wheel.urdf.xacro (robot description, xacro)
@@ -32,6 +32,6 @@
 			</visual>
 			<collision>
-				<origin xyz="0 ${reflect_link_y * -0.012} 0" rpy="${PI/2} 0 0" /> <geometry> <cylinder length="${simple_wheel_length}" radius="${simple_wheel_radius}"/> </geometry>
-<!-- 				<origin xyz="0 ${reflect_link_y * wheel_origin_y} 0" rpy="0 0 ${origin_yaw}" /> <geometry> <mesh filename="package://guardian_description/meshes/wheel.stl" /> </geometry> -->
+<!-- 				<origin xyz="0 ${reflect_link_y * -0.012} 0" rpy="${PI/2} 0 0" /> <geometry> <cylinder length="${simple_wheel_length}" radius="${simple_wheel_radius}"/> </geometry> -->
+				<origin xyz="0 ${reflect_link_y * wheel_origin_y} 0" rpy="0 0 ${origin_yaw}" /> <geometry> <mesh filename="package://guardian_description/meshes/wheel.stl" /> </geometry>
 			</collision>
 		</link>
