Commit message: Improved simulation of robot tracks in gazebo (now instead of 5 it has 12 wheels following the underside of each track).

File: guardian_sim/guardian_description/urdf/guardian_tracks.urdf.xacro (robot description, xacro)
@@ -6,5 +6,5 @@
 	<!-- args: useSimulatedKinect useSchunkArm publishOdometryTf publishOdometryMsg -->
 	<!-- ###### BASE ###### -->
-	<guardian_base base_footprint_z="0.0635" use_simulated_kinect="$(arg useSimulatedKinect)" use_schunk_arm="$(arg useSchunkArm)" use_planar_lasers="$(arg usePlanarLasers) />
+	<guardian_base base_footprint_z="0.0635" use_simulated_kinect="$(arg useSimulatedKinect)" use_schunk_arm="$(arg useSchunkArm)" use_planar_lasers="$(arg usePlanarLasers)" />
 	<!-- ###### TRACKS ###### -->
 	<!-- visual -->
@@ -12,15 +12,31 @@
 	<track parent="base_link" prefix="right_track" joint_yaw="0" />
 	<!-- right track collision -->
-	<track_wheel parent="right_track" prefix="right_tw_1" origin_yaw="0" wheel_offset_x="0.3" reflect_y="-1" joint_yaw="0" />
-	<track_wheel parent="right_track" prefix="right_tw_2" origin_yaw="0" wheel_offset_x="0.15" reflect_y="-1" joint_yaw="0" />
-	<track_wheel parent="right_track" prefix="right_tw_3" origin_yaw="0" wheel_offset_x="0" reflect_y="-1" joint_yaw="0" />
-	<track_wheel parent="right_track" prefix="right_tw_4" origin_yaw="0" wheel_offset_x="-0.15" reflect_y="-1" joint_yaw="0" />
-	<track_wheel parent="right_track" prefix="right_tw_5" origin_yaw="0" wheel_offset_x="-0.3" reflect_y="-1" joint_yaw="0" />
+	<track_wheel parent="right_track" prefix="right_tw_0"  origin_yaw="0" wheel_offset_x="0.43"   wheel_offset_z="0.103"  reflect_y="-1" joint_yaw="0" wheel_radius="0.13"   wheel_length="0.05" />
+	<track_wheel parent="right_track" prefix="right_tw_1"  origin_yaw="0" wheel_offset_x="0.375"  wheel_offset_z="0.0945" reflect_y="-1" joint_yaw="0" wheel_radius="0.1375" wheel_length="0.05" />
+	<track_wheel parent="right_track" prefix="right_tw_2"  origin_yaw="0" wheel_offset_x="0.3"    wheel_offset_z="0.086"  reflect_y="-1" joint_yaw="0" wheel_radius="0.147"  wheel_length="0.05" />
+	<track_wheel parent="right_track" prefix="right_tw_3"  origin_yaw="0" wheel_offset_x="0.225"  wheel_offset_z="0.081"  reflect_y="-1" joint_yaw="0" wheel_radius="0.15"   wheel_length="0.05" />
+	<track_wheel parent="right_track" prefix="right_tw_4"  origin_yaw="0" wheel_offset_x="0.15"   wheel_offset_z="0.081"  reflect_y="-1" joint_yaw="0" wheel_radius="0.15"   wheel_length="0.05" />
+	<track_wheel parent="right_track" prefix="right_tw_5"  origin_yaw="0" wheel_offset_x="0.075"  wheel_offset_z="0.081"  reflect_y="-1" joint_yaw="0" wheel_radius="0.15"   wheel_length="0.05" />
+	<track_wheel parent="right_track" prefix="right_tw_6"  origin_yaw="0" wheel_offset_x="0"      wheel_offset_z="0.081"  reflect_y="-1" joint_yaw="0" wheel_radius="0.15"   wheel_length="0.05" />
+	<track_wheel parent="right_track" prefix="right_tw_7"  origin_yaw="0" wheel_offset_x="-0.075" wheel_offset_z="0.081"  reflect_y="-1" joint_yaw="0" wheel_radius="0.15"   wheel_length="0.05" />
+	<track_wheel parent="right_track" prefix="right_tw_8"  origin_yaw="0" wheel_offset_x="-0.15"  wheel_offset_z="0.081"  reflect_y="-1" joint_yaw="0" wheel_radius="0.15"   wheel_length="0.05" />
+	<track_wheel parent="right_track" prefix="right_tw_9"  origin_yaw="0" wheel_offset_x="-0.225" wheel_offset_z="0.081"  reflect_y="-1" joint_yaw="0" wheel_radius="0.15"   wheel_length="0.05" />
+	<track_wheel parent="right_track" prefix="right_tw_10" origin_yaw="0" wheel_offset_x="-0.3"   wheel_offset_z="0.086"  reflect_y="-1" joint_yaw="0" wheel_radius="0.147"  wheel_length="0.05" />
+	<track_wheel parent="right_track" prefix="right_tw_11" origin_yaw="0" wheel_offset_x="-0.375" wheel_offset_z="0.0945" reflect_y="-1" joint_yaw="0" wheel_radius="0.1375" wheel_length="0.05" />
+	<track_wheel parent="right_track" prefix="right_tw_12" origin_yaw="0" wheel_offset_x="-0.43"  wheel_offset_z="0.103"  reflect_y="-1" joint_yaw="0" wheel_radius="0.13"   wheel_length="0.05" />
 	<!-- left track collision -->
-	<track_wheel parent="left_track" prefix="left_tw_1" origin_yaw="${PI}" wheel_offset_x="0.3" reflect_y="-1" joint_yaw="${PI}" />
-	<track_wheel parent="left_track" prefix="left_tw_2" origin_yaw="0" wheel_offset_x="0.15" reflect_y="-1" joint_yaw="${PI}" />
-	<track_wheel parent="left_track" prefix="left_tw_3" origin_yaw="0" wheel_offset_x="0" reflect_y="-1" joint_yaw="${PI}" />
-	<track_wheel parent="left_track" prefix="left_tw_4" origin_yaw="0" wheel_offset_x="-0.15" reflect_y="-1" joint_yaw="${PI}" />
-	<track_wheel parent="left_track" prefix="left_tw_5" origin_yaw="0" wheel_offset_x="-0.3" reflect_y="-1" joint_yaw="${PI}" />
+	<track_wheel parent="left_track" prefix="left_tw_0"    origin_yaw="0" wheel_offset_x="0.43"   wheel_offset_z="0.103"  reflect_y="-1" joint_yaw="${PI}" wheel_radius="0.13"   wheel_length="0.05" />
+	<track_wheel parent="left_track" prefix="left_tw_1"    origin_yaw="0" wheel_offset_x="0.375"  wheel_offset_z="0.0945" reflect_y="-1" joint_yaw="${PI}" wheel_radius="0.1375" wheel_length="0.05" />
+	<track_wheel parent="left_track" prefix="left_tw_2"    origin_yaw="0" wheel_offset_x="0.3"    wheel_offset_z="0.086"  reflect_y="-1" joint_yaw="${PI}" wheel_radius="0.147"  wheel_length="0.05" />
+	<track_wheel parent="left_track" prefix="left_tw_3"    origin_yaw="0" wheel_offset_x="0.225"  wheel_offset_z="0.081"  reflect_y="-1" joint_yaw="${PI}" wheel_radius="0.15"   wheel_length="0.05" />
+	<track_wheel parent="left_track" prefix="left_tw_4"    origin_yaw="0" wheel_offset_x="0.15"   wheel_offset_z="0.081"  reflect_y="-1" joint_yaw="${PI}" wheel_radius="0.15"   wheel_length="0.05" />
+	<track_wheel parent="left_track" prefix="left_tw_5"    origin_yaw="0" wheel_offset_x="0.075"  wheel_offset_z="0.081"  reflect_y="-1" joint_yaw="${PI}" wheel_radius="0.15"   wheel_length="0.05" />
+	<track_wheel parent="left_track" prefix="left_tw_6"    origin_yaw="0" wheel_offset_x="0"      wheel_offset_z="0.081"  reflect_y="-1" joint_yaw="${PI}" wheel_radius="0.15"   wheel_length="0.05" />
+	<track_wheel parent="left_track" prefix="left_tw_7"    origin_yaw="0" wheel_offset_x="-0.075" wheel_offset_z="0.081"  reflect_y="-1" joint_yaw="${PI}" wheel_radius="0.15"   wheel_length="0.05" />
+	<track_wheel parent="left_track" prefix="left_tw_8"    origin_yaw="0" wheel_offset_x="-0.15"  wheel_offset_z="0.081"  reflect_y="-1" joint_yaw="${PI}" wheel_radius="0.15"   wheel_length="0.05" />
+	<track_wheel parent="left_track" prefix="left_tw_9"    origin_yaw="0" wheel_offset_x="-0.225" wheel_offset_z="0.081"  reflect_y="-1" joint_yaw="${PI}" wheel_radius="0.15"   wheel_length="0.05" />
+	<track_wheel parent="left_track" prefix="left_tw_10"   origin_yaw="0" wheel_offset_x="-0.3"   wheel_offset_z="0.086"  reflect_y="-1" joint_yaw="${PI}" wheel_radius="0.147"  wheel_length="0.05" />
+	<track_wheel parent="left_track" prefix="left_tw_11"   origin_yaw="0" wheel_offset_x="-0.375" wheel_offset_z="0.0945" reflect_y="-1" joint_yaw="${PI}" wheel_radius="0.1375" wheel_length="0.05" />
+	<track_wheel parent="left_track" prefix="left_tw_12"   origin_yaw="0" wheel_offset_x="-0.43"  wheel_offset_z="0.103"  reflect_y="-1" joint_yaw="${PI}" wheel_radius="0.13"   wheel_length="0.05" />
 	<!-- ###### PLUGIN ###### -->
 	<gazebo> <!-- from hector_gazebo -->
@@ -28,9 +44,9 @@
 			<alwaysOn>true</alwaysOn>
 			<updateRate>10.0</updateRate>
-			<leftJoints>joint_left_tw_1 joint_left_tw_2 joint_left_tw_3 joint_left_tw_4 joint_left_tw_5 </leftJoints>
-			<rightJoints>joint_right_tw_1 joint_right_tw_2 joint_right_tw_3 joint_right_tw_4 joint_right_tw_5 </rightJoints>
+			<leftJoints>joint_left_tw_0 joint_left_tw_1 joint_left_tw_2 joint_left_tw_3 joint_left_tw_4 joint_left_tw_5 joint_left_tw_6 joint_left_tw_7 joint_left_tw_8 joint_left_tw_9 joint_left_tw_10 joint_left_tw_11 joint_left_tw_12</leftJoints>
+			<rightJoints>joint_right_tw_0 joint_right_tw_1 joint_right_tw_2 joint_right_tw_3 joint_right_tw_4 joint_right_tw_5 joint_right_tw_6 joint_right_tw_7 joint_right_tw_8 joint_right_tw_9 joint_right_tw_10 joint_right_tw_11 joint_right_tw_12</rightJoints>
 			<wheelSeparation>0.448</wheelSeparation>
 			<wheelDiameter>0.3</wheelDiameter>
-			<torque>20</torque>
+			<torque>60</torque>
 			<robotBaseFrame>base_footprint</robotBaseFrame>
 			<commandTopic>/guardian/cmd_vel</commandTopic>

File: guardian_sim/guardian_description/urdf/track_wheel.urdf.xacro (robot description, xacro)
@@ -7,5 +7,5 @@
 	<!-- <xacro:property name="wheel_origin_y" value="0.0" /> -->
 	<xacro:property name="wheel_offset_y" value="0.224" />
-	<xacro:property name="wheel_offset_z" value="0.081" /> <!-- 0.15-0.069 -->
+<!-- 	<xacro:property name="wheel_offset_z" value="0.081" /> 0.15-0.069 -->
 	<xacro:property name="wheel_joint_damping" value="0.0" />
 	<xacro:property name="wheel_joint_friction" value="0.0" />
@@ -13,5 +13,5 @@
 	<xacro:property name="wheel_joint_velocity_limit" value="200.0" />
 	<xacro:property name="wheel_mechanical_reduction" value="1.0" />
-	<xacro:macro name="track_wheel" params="parent prefix origin_yaw wheel_offset_x reflect_y joint_yaw">
+	<xacro:macro name="track_wheel" params="parent prefix origin_yaw wheel_offset_x wheel_offset_z reflect_y joint_yaw wheel_radius wheel_length">
 		<link name="${prefix}">
 			<inertial>
@@ -22,12 +22,12 @@
 				<!-- iyy="0.00015218160428" iyz="0.0" -->
 				<!-- izz="0.00011763977943" /> -->
-				<!-- <inertia ixx="${(1/12)*mass*(3*simple_wheel_radius * simple_wheel_radius + simple_wheel_length*simple_wheel_length)}" ixy="0.0" ixz="0.0" -->
-				<!-- iyy="${(1/12)*mass*(3*simple_wheel_radius * simple_wheel_radius + simple_wheel_length*simple_wheel_length)}" iyz="0.0" -->
-				<!-- izz="${0.5*mass*(simple_wheel_radius * simple_wheel_radius)}" /> wikipedia formula -->
+				<!-- <inertia ixx="${(1/12)*mass*(3*wheel_radius * wheel_radius + wheel_length*wheel_length)}" ixy="0.0" ixz="0.0" -->
+				<!-- iyy="${(1/12)*mass*(3*wheel_radius * wheel_radius + wheel_length*wheel_length)}" iyz="0.0" -->
+				<!-- izz="${0.5*mass*(wheel_radius * wheel_radius)}" /> wikipedia formula -->
 			</inertial>
 			<!-- <visual> -->
 			<!-- <origin xyz="0 ${reflect_y * wheel_origin_y} 0" rpy="${PI/2} 0 ${origin_yaw}" /> -->
 			<!-- <geometry> -->
-			<!-- <cylinder length="${simple_wheel_length}" radius="${simple_wheel_radius}"/> -->
+			<!-- <cylinder length="${wheel_length}" radius="${wheel_radius}"/> -->
 			<!-- </geometry> -->
 			<!-- <material name="black"> -->
@@ -38,5 +38,5 @@
 				<origin xyz="0 0 0" rpy="${PI/2} 0 ${origin_yaw}" />
 				<geometry>
-					<cylinder length="${simple_wheel_length}" radius="${simple_wheel_radius}" />
+					<cylinder length="${wheel_length}" radius="${wheel_radius}" />
 				</geometry>
 				<!-- <material name="black"/> -->
@@ -53,5 +53,7 @@
 		<transmission name="joint_${prefix}_trans">
 			<type>transmission_interface/SimpleTransmission</type>
-			<joint name="joint_${prefix}" />
+			<joint name="joint_${prefix}">
+				<hardwareInterface>EffortJointInterface</hardwareInterface>
+			</joint>
 			<actuator name="joint_${prefix}_motor">
 				<hardwareInterface>EffortJointInterface</hardwareInterface>
