Commit message: Synced link/joint names of robot with the gazebo simulation.

File: guardian_sim/guardian_description/urdf/sensors/hokuyo_front.urdf.xacro (robot description, xacro)
@@ -43,5 +43,7 @@
 		<transmission name="joint_${prefix}_trans">
 			<type>transmission_interface/SimpleTransmission</type>
-			<joint name="hokuyo_${prefix}_joint" />
+			<joint name="hokuyo_${prefix}_tilt_joint" >
+				<hardwareInterface>EffortJointInterface</hardwareInterface>
+			</joint>
 			<actuator name="${prefix}_motor">
 				<hardwareInterface>EffortJointInterface</hardwareInterface>

File: guardian_sim/guardian_description/urdf/sensors/imu.urdf.xacro (robot description, xacro)
@@ -40,9 +40,9 @@
 			</plugin>
 		</gazebo>
-		<link name="imu_um7_link" />
-		<joint name="imu_um7_joint" type="fixed">
+		<link name="imu_link" />
+		<joint name="imu_joint" type="fixed">
 			<origin xyz="0.056 0.0 0.1355" rpy="0 0 0 " />
 			<parent link="${parent}" />
-			<child link="imu_um7_link" />
+			<child link="imu_link" />
 		</joint>
 	</xacro:macro>

File: guardian_sim/guardian_description/urdf/wheel.urdf.xacro (robot description, xacro)
@@ -46,5 +46,7 @@
 		<transmission name="joint_${prefix}_trans">
 			<type>transmission_interface/SimpleTransmission</type>
-			<joint name="joint_${prefix}_wheel" />
+			<joint name="joint_${prefix}_wheel" >
+				<hardwareInterface>EffortJointInterface</hardwareInterface>
+			</joint>
 			<actuator name="joint_${prefix}_motor">
 				<hardwareInterface>EffortJointInterface</hardwareInterface>
